File: front panel/Original with 9602/front panel 9602.sch (KiCad schematic (older format))
At the start: 163 parts, among them J1 Accumulator, J10 Conn_01x04_Female, J11 Conn_01x04_Female, J12 Conn_01x04_Female, J13 ~EXT.LA, J14 Z-BIT, J2 Mem_Buffer, J3 Conn_01x16_Female, J4 Conn_01x04_Female, J5 Conn_01x04_Female, J6 Conn_01x04_Female, J7 SR_REGISTER, J8 Conn_01x04_Female, J9 Conn_01x04_Female, SW1 SR0, SW10 DEPOSIT, SW11 EXAM, SW12 RUN, SW13 HALT, SW14 SINGLE, SW15 SLOW, SW16 CP, SW2 SR1, SW3 SR2, SW4 SR3, SW5 SR4, SW6 SR5, SW7 SR6, SW8 SR7, SW9 LD_ADD, U1 74LS05, U10 74LS123, U11 74LS05, U12 7400, U2 74LS05, U3 74LS05, U4 7417, U5 7417, U6 7400, U7 74LS05, U8 7400, U9 7400

Commit message: New PCB with all the corrections made
Parts:
- C1, C6, C7, C8: symbol Device:C_Small -> front-panel-9602-rescue:C_Small-Device
- C2: symbol Device:CP_Small -> front-panel-9602-rescue:CP_Small-Device
- C3, C4, C5: symbol Device:C -> front-panel-9602-rescue:C-Device
- D1, D10, D11, D12, D13, D14, D15, D16, D17, D18, D19, D2, D20, D21, D22, D23, D24, D25, D26, D27, D28, D29, D3, D30, D31, D32, D33, D34, D35, D36, D37, D38, D39, D4, D40, D41, D42, D43, D44, D5, D6, D7, D8, D9: symbol Device:LED -> front-panel-9602-rescue:LED-Device
- H1, H3, H5: symbol Mechanical:MountingHole -> front-panel-9602-rescue:MountingHole-Mechanical
- H2, H4, H6: symbol Mechanical:MountingHole_Pad -> front-panel-9602-rescue:MountingHole_Pad-Mechanical
- J1, J2, J7: symbol Connector:Conn_01x08_Female -> front-panel-9602-rescue:Conn_01x08_Female-Connector
- J10, J11, J12, J4, J5, J6, J8, J9: symbol Connector:Conn_01x04_Female -> front-panel-9602-rescue:Conn_01x04_Female-Connector
- J13, J14: symbol Connector:Conn_01x01_Female -> front-panel-9602-rescue:Conn_01x01_Female-Connector
- J3: symbol Connector:Conn_01x16_Female -> front-panel-9602-rescue:Conn_01x16_Female-Connector
- R1, R10, R11, R12, R13, R14, R15, R16, R17, R18, R19, R2, R20, R21, R22, R23, R24, R25, R26, R27, R28, R29, R3, R30, R31, R32, R33, R34, R35, R36, R37, R38, R39, R4, R40, R41, R42, R43, R44, R45, R46, R47, R48, R49, R5, R50, R51, R53, R54, R55, R56, R57, R58, R59, R6, R60, R63, R7, R8, R9: symbol Device:R_Small -> front-panel-9602-rescue:R_Small-Device
- R52, R61, R62: symbol Device:R -> front-panel-9602-rescue:R-Device
- SW1, SW10, SW11, SW12, SW13, SW14, SW15, SW16, SW2, SW3, SW4, SW5, SW6, SW7, SW8, SW9: symbol Switch:SW_DPDT_x2 -> front-panel-9602-rescue:SW_DPDT_x2-Switch
- U1, U11, U2, U3, U7: symbol 74xx:74LS05 -> front-panel-9602-rescue:74LS05-74xx
- U10: symbol 74xx:74LS123 -> front-panel-9602-rescue:74LS123-74xx
- U12, U6, U8, U9: symbol 74xx:7400 -> front-panel-9602-rescue:7400-74xx
- U4, U5: symbol front-panel-9602-rescue:7417-74xx-front-panel-rescue -> front-panel-9602-rescue:7417-74xx-front-panel-rescue-front-panel-9602-rescue
