File: front panel/Original with 9602/front panel 9602.kicad_pcb (KiCad board)
At the start: 2 copper layers, 283 x 96 mm, 165 parts, among them J1 Accumulator, J10 Conn_01x04_Female, J11 Conn_01x04_Female, J12 Conn_01x04_Female, J13 ~EXT.LA, J14 Z-BIT, J2 Mem_Buffer, J3 Conn_01x16_Female, J4 Conn_01x04_Female, J5 Conn_01x04_Female, J6 Conn_01x04_Female, J7 SR_REGISTER, J8 Conn_01x04_Female, J9 Conn_01x04_Female, SW1 SR0, SW10 DEPOSIT, SW11 HALT, SW12 SINGLE, SW13 F/S, SW14 PAGE ZERO, SW15 RUN, SW16 EXAM, SW2 SR1, SW3 SR2, SW4 SR3, SW5 SR4, SW6 SR5, SW7 SR6, SW8 SR7, SW9 LD_ADDR, U1 74LS05, U10 DM9602, U11 74LS05, U12 74LS00, U2 74LS05, U3 74LS05, U4 74LS07, U5 74LS07, U6 74LS00, U7 74LS05, U8 74LS00, U9 74LS00

Commit message: New PCB with all the corrections made
Parts:
- added H3: MountingHole, MountingHole:MountingHole_3.2mm_M3, F.Cu at (144.6, 190.7)
- SW1: value SR0 -> 0; footprint dBSound_library:DPDT_toggle_switch_wired -> EDUC-8:SPDT_toggle_switch_wired
- SW2: value SR1 -> 1; footprint dBSound_library:DPDT_toggle_switch_wired -> EDUC-8:SPDT_toggle_switch_wired
- SW3: value SR2 -> 2; footprint dBSound_library:DPDT_toggle_switch_wired -> EDUC-8:SPDT_toggle_switch_wired
- SW4: value SR3 -> 3; footprint dBSound_library:DPDT_toggle_switch_wired -> EDUC-8:SPDT_toggle_switch_wired
- SW5: value SR4 -> 4; footprint dBSound_library:DPDT_toggle_switch_wired -> EDUC-8:SPDT_toggle_switch_wired
- SW6: value SR5 -> 5; footprint dBSound_library:DPDT_toggle_switch_wired -> EDUC-8:SPDT_toggle_switch_wired
- SW7: value SR6 -> 6; footprint dBSound_library:DPDT_toggle_switch_wired -> EDUC-8:SPDT_toggle_switch_wired
- SW8: value SR7 -> 7; footprint dBSound_library:DPDT_toggle_switch_wired -> EDUC-8:SPDT_toggle_switch_wired
- moved R59 19.2 mm to (218.2, 128.3), turned to 90 degrees
- moved SW1 1.26 mm to (172.0, 123.4), turned to 0 degrees
- moved SW3 1.26 mm to (144.4, 123.4), turned to 0 degrees
- moved SW5 1.26 mm to (116.8, 123.4), turned to 0 degrees
- moved SW8 1.26 mm to (75.4, 123.4), turned to 0 degrees
- moved SW4 1.26 mm to (130.6, 123.4), turned to 0 degrees
- moved SW6 1.26 mm to (103.0, 123.4), turned to 0 degrees
- moved SW7 1.26 mm to (89.2, 123.4), turned to 0 degrees
- moved SW2 1.26 mm to (158.2, 123.4), turned to 0 degrees
Connections:
- U10 pad 9: (no net) -> ~{RUN_COMMAND}
Routing:
- net +5V: track 797.0 -> 891.5 mm
- net GND: track 930.8 -> 899.2 mm
- net Net-(R59-Pad1): track 88.4 -> 68.1 mm
- net SR1: track 37.9 -> 23.4 mm
- net SR5: track 79.7 -> 65.9 mm
- net SR2: track 45.9 -> 32.8 mm
- net SR3: track 56.4 -> 43.4 mm
- net SR4: track 67.6 -> 55.0 mm
- net SR0: track 43.7 -> 32.4 mm
- net SR7: track 106.3 -> 96.1 mm
- net SR6: track 95.3 -> 85.1 mm
- net ~{RUN_COMMAND}: track 0.00 -> 8.98 mm
- net ~{EXT.LA}: track 341.3 -> 343.8 mm
Other:
- board text removed: "ʕ •ᴥ•ʔ"

Commit message: Schematic update 2024-04-14 plus fixes
Parts:
- J14: value Z-BIT -> Conn_01x02_Male; footprint Connector_PinSocket_2.54mm:PinSocket_1x01_P2.54mm_Vertical -> Connector_JST:JST_XH_B2B-XH-A_1x02_P2.50mm_Vertical; moved to F.Cu
- moved J14 40.4 mm to (196.0, 112.7)
- moved R40 3.28 mm to (279.4, 67.7)
- moved R24 3.03 mm to (90.8, 51.8)
- moved R50 2.94 mm to (109.6, 120.8)
- moved R15 2.90 mm to (90.8, 47.9)
- moved R49 2.84 mm to (123.7, 120.6)
- moved R51 2.72 mm to (86.2, 113.6)
- moved R36 2.67 mm to (246.7, 67.6)
- moved R47 2.66 mm to (151.2, 120.5)
- moved R33 2.57 mm to (241.5, 67.7)
- moved R35 2.57 mm to (262.7, 67.7)
- moved R37 2.57 mm to (266.8, 67.7)
- moved R34 2.55 mm to (251.7, 67.6)
- moved R10 2.55 mm to (173.0, 58.7)
- moved R48 2.54 mm to (136.3, 120.6)
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Connections:
- J14 pad 1: Net-(J14-Pad1) -> Net-(SW14-Pad2)
- SW14 pad 2: Net-(J14-Pad1) -> Net-(SW14-Pad2)
Routing:
- net +5V: track 891.5 -> 939.6 mm
- net Net-(J14-Pad1): track 41.9 -> 0.00 mm
- net GND: track 899.2 -> 922.2 mm
- net Net-(SW14-Pad2): track 0.00 -> 18.2 mm
- net Net-(D40-Pad1): track 105.9 -> 100.9 mm
- net Net-(D18-Pad1): track 50.4 -> 54.6 mm
- net Net-(R35-Pad1): track 27.7 -> 23.6 mm
- net ~{DEPOSIT}: track 71.5 -> 67.4 mm
- net MA4: track 26.0 -> 22.1 mm
- net Net-(D16-Pad1): track 18.1 -> 21.6 mm
- net ~{JMS}: track 12.7 -> 16.1 mm
- net Net-(U6-Pad2): track 106.1 -> 102.8 mm
- net Net-(R40-Pad1): track 8.24 -> 5.04 mm
- net Net-(D9-Pad1): track 26.7 -> 29.8 mm
- net MA7: track 66.3 -> 63.2 mm
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Other:
- board text added: "Designed by Jamieson Rowe Electronics Australia 1974 PCB by Gwyllym Suter 2024"
- board text removed: "Designed by Jamieson Rowe Electronics Australia 1974 PCB by Gwyllym Suter"
- board text removed: "V1.1"
