File: Decoder/educ 8 decoder.sch (KiCad schematic (older format))
At the start: 26 parts, among them J1 32-way-pcb-edge-Educ-8-connec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, J2 16-way-pcb-edge-Educ-8-connec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, U1 74LS00, U10 74LS00, U11 74LS00, U12 74LS00, U13 74LS00, U14 74LS04, U2 74LS10, U3 74LS04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

Commit message: Schematic update 2024-04-14 plus fixes
Parts:
- C1, C10, C11, C12, C2, C4: symbol Device:C -> educ-8-decoder-rescue:C-Device
- H1, H2: symbol educ-8-decoder-rescue:Card_handle-EDUC-8 -> educ-8-decoder-rescue:Card_handle-EDUC-8-educ-8-decoder-rescue
- J1: symbol educ-8-decoder-rescue:32-way-pcb-edge-Educ-8-connectors-EDUC-8 -> educ-8-decoder-rescue:32-way-pcb-edge-Educ-8-connectors-EDUC-8-educ-8-decoder-rescue
- J2: symbol educ-8-decoder-rescue:16-way-pcb-edge-Educ-8-connectors-EDUC-8 -> educ-8-decoder-rescue:16-way-pcb-edge-Educ-8-connectors-EDUC-8-educ-8-decoder-rescue
- R1, R2: symbol Device:R -> educ-8-decoder-rescue:R-Device
Changed lines of the file:
@@
 	14200 5300 13450 5300
 $Comp
-L Device:R R1
+L educ-8-decoder-rescue:R-Device R1
 U 1 1 5D801CC1
 P 13950 5500
@@
 	13250 5500 13250 5400
 $Comp
-L power:+5V #PWR0101
+L educ-8-decoder-rescue:+5V-power #PWR0101
 U 1 1 5D8172F0
 P 13250 5400
@@
 	12700 11800 12200 11800
 $Comp
-L power:+5V #PWR0102
+L educ-8-decoder-rescue:+5V-power #PWR0102
 U 1 1 5E4BD966
 P 7950 11700
@@
 $EndComp
 $Comp
-L power:+5V #PWR0103
+L educ-8-decoder-rescue:+5V-power #PWR0103
 U 1 1 5E4BFA49
 P 4450 3650
@@
 $EndComp
 $Comp
-L power:GND #PWR0104
+L educ-8-decoder-rescue:GND-power #PWR0104
 U 1 1 5E4C0D34
 P 8000 14000
@@
 $EndComp
 $Comp
-L power:GND #PWR0105
+L educ-8-decoder-rescue:GND-power #PWR0105
 U 1 1 5E4C2DDC
 P 4450 5250
@@
 	8000 13850 8750 13850
 $Comp
-L Device:C C1
+L educ-8-decoder-rescue:C-Device C1
 U 1 1 5F2D4A65
 P 1900 12100
@@
 $EndComp
 $Comp
-L power:GND #PWR0108
+L educ-8-decoder-rescue:GND-power #PWR0108
 U 1 1 5F2D6A7C
 P 1900 12400
@@
 	1900 12250 1900 12400
 $Comp
-L Device:C C2
+L educ-8-decoder-rescue:C-Device C2
 U 1 1 5F34792E
 P 2850 12100
@@
 $EndComp
 $Comp
-L power:GND #PWR0109
+L educ-8-decoder-rescue:GND-power #PWR0109
 U 1 1 5F347934
 P 2850 12400
@@
 	2850 12250 2850 12400
 $Comp
-L Device:C C4
+L educ-8-decoder-rescue:C-Device C4
 U 1 1 5F38F9B9
 P 4700 12100
@@
 $EndComp
 $Comp
-L power:GND #PWR0111
+L educ-8-decoder-rescue:GND-power #PWR0111
 U 1 1 5F38F9BF
 P 4700 12400
@@
 	4700 12250 4700 12400
 $Comp
-L Device:C C10
+L educ-8-decoder-rescue:C-Device C10
 U 1 1 5F5643FB
 P 10250 12100
@@
 $EndComp
 $Comp
-L power:GND #PWR0116
+L educ-8-decoder-rescue:GND-power #PWR0116
 U 1 1 5F564401
 P 10250 12400
@@
 	10250 12250 10250 12400
 $Comp
-L Device:C C11
+L educ-8-decoder-rescue:C-Device C11
 U 1 1 5F588DA0
 P 11200 12100
@@
 $EndComp
 $Comp
-L power:GND #PWR0117
+L educ-8-decoder-rescue:GND-power #PWR0117
 U 1 1 5F588DA6
 P 11200 12400
@@
 	11200 12250 11200 12400
 $Comp
-L Device:C C12
+L educ-8-decoder-rescue:C-Device C12
 U 1 1 5F5ADA72
 P 12200 12100
@@
 $EndComp
 $Comp
-L power:GND #PWR0118
+L educ-8-decoder-rescue:GND-power #PWR0118
 U 1 1 5F5ADA78
 P 12200 12400
@@
 GND
 $Comp
-L educ-8-decoder-rescue:32-way-pcb-edge-Educ-8-connectors-EDUC-8 J1
+L educ-8-decoder-rescue:32-way-pcb-edge-Educ-8-connectors-EDUC-8-educ-8-decoder-rescue J1
 U 1 1 60B6130C
 P 17000 9700
@@
 $EndComp
 $Comp
-L educ-8-decoder-rescue:16-way-pcb-edge-Educ-8-connectors-EDUC-8 J2
+L educ-8-decoder-rescue:16-way-pcb-edge-Educ-8-connectors-EDUC-8-educ-8-decoder-rescue J2
 U 1 1 60C0F5B3
 P 17000 12550
@@
 Connection ~ 6200 8450
 $Comp
-L Device:R R2
+L educ-8-decoder-rescue:R-Device R2
 U 1 1 61545921
 P 3750 4050
@@
 $EndComp
 $Comp
-L power:+5V #PWR01
+L educ-8-decoder-rescue:+5V-power #PWR01
 U 1 1 61546A9E
 P 3500 4000
@@
 T0.5
 $Comp
-L educ-8-decoder-rescue:Card_handle-EDUC-8 H1
+L educ-8-decoder-rescue:Card_handle-EDUC-8-educ-8-decoder-rescue H1
 U 1 1 61C6081F
 P 20100 10150
@@
 $EndComp
 $Comp
-L educ-8-decoder-rescue:Card_handle-EDUC-8 H2
+L educ-8-decoder-rescue:Card_handle-EDUC-8-educ-8-decoder-rescue H2
 U 1 1 61C60BCA
 P 21500 10150
@@
 	6150 11800 7200 11800
 $Comp
-L power:GND #PWR0106
+L educ-8-decoder-rescue:GND-power #PWR0106
 U 1 1 62C7CD81
 P 20900 10400
