File: Decoder/educ 8 decoder.kicad_sch (KiCad schematic)
At the start: 26 parts, among them J1 32-way-pcb-edge-Educ-8-connec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, J2 16-way-pcb-edge-Educ-8-connec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, U1 74LS00, U10 74LS00, U11 74LS00, U12 74LS00, U13 74LS00, U14 74LS04, U2 74LS10, U3 74LS04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

Commit message: Schematic update 2024-04-14 plus fixes
Other:
- note added: "C1 47nF C2 47nF C4 47nF C10 47nF C11 47nF C12 47nF H1 Card_handle H2 Card_handle J1 32-way-pcb-edge connector J2 16-way-pcb-edge-connector R1 2K2 R2 2K2 U1 74LS00 U2 74LS10 U3 74LS04 U4 74LS10 U5 74LS00 U6 74LS20 U7 74LS00 U8 74LS259 U9 74LS00 U10 74LS00 U11 74LS00 U12 74LS00 U13 74LS00 U14 74LS04"
- note removed: "100nF 50v Polyester"
- note removed: "100uF 35v electro"
- note removed: "2.2K 1/4 Watt resistor"
- note removed: "3 input NAND"
- note removed: "4 input NAND"
- note removed: "74LS00"
- note removed: "74LS04"
- note removed: "74LS10"
- note removed: "74LS20"
- note removed: "74LS259"
- note removed: "Addressable 8 bit latch"
- note removed: "C1"
- note removed: "C1-14"
- note removed: "C10"
- note removed: "C11"
- note removed: "C12"
- note removed: "C13"
- note removed: "C14"
- note removed: "C15"
- note removed: "C15-16"
- note removed: "C16"
- note removed: "C2"
- note removed: "C3"
- note removed: "C4"
- note removed: "C5"
- note removed: "C6"
- note removed: "C7"
- note removed: "C8"
- note removed: "C9"
- note removed: "Hex Inverter"
- note removed: "QTY"
- note removed: "Quad NAND"
- note removed: "R1"
- note removed: "RefDes"
- note removed: "Supplier"
- note removed: "T0.5 and T22.5 were flipped. change them around as shown"
- note removed: "Type"
- note removed: "U1"
- note removed: "U10"
- note removed: "U11"
- note removed: "U12"
- note removed: "U13"
- note removed: "U3"
- note removed: "U5"
- note removed: "U6"
- note removed: "U7"
- note removed: "U8"
- note removed: "U9"
- note removed: "“"

Commit message: Changes 20-7-2025 E8/T. Connected 3 missing supply rail tracks to ICS Added flood fill top and bottom to reduce noise E8/F Corrected labelling on RHS board to reflect EXT_LA not GND Changed fast slow switch operation so fast is in the DOWN position. E8/C. Ran a new track to the 2 pin JST connector from EXT_LA from 10 pin connector on SR input. Added files for E8MX, 2k byte memory expansion board
Parts:
- U13: footprint Package_DIP:DIP-14_W7.62mm_LongPads -> iot_shift
Connections:
- net FETCH: now also U13.1; no longer U13.2
- net T0.5: now also U13.2; no longer U13.5
- net T22.5: now also U13.5; no longer U13.1
Other:
- note added: "1. When using LS series replace R1 and R2 with a wire link"
- note added: "Install link for LS series"
- note added: "Install wire link for LS series"
- note added: "~{DEFER}"
- note removed: "1. Inputs for all unused gates connected to GND"
- note removed: "Every track and pad checked against the original artwork"
- note removed: "~{DEFER }"
- moved on the sheet: U14F
