File: Input:Output Interface/Input:Output Interface.sch (KiCad schematic (older format))
At the start: 25 parts, among them J1 Conn_01x03_Male, J2 Conn_01x03_Male, J3 16-way-pcb-edge-Educ-8-connec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, J4 16-way-pcb-edge-Educ-8-connec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, U1 74LS37, U10 74LS01, U11 74LS04, U2 74LS04, U3 7400, U4 74LS04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

Commit message: Schematic update 2024-04-14 plus fixes
Parts:
- C1, C2, C3, C4: symbol Device:C -> Input:Output-Interface-rescue_Output-Interface-rescue_C-Device-Input
- H1, H2: symbol EDUC-8:Card_handle -> Input:Output-Interface-rescue_Output-Interface-rescue_Card_handle-EDUC-8-Input
- J1, J2: symbol Connector:Conn_01x03_Male -> Input:Output-Interface-rescue_Output-Interface-rescue_Conn_01x03_Male-Connector-Input
- J3, J4: symbol EDUC-8:16-way-pcb-edge-Educ-8-connectors -> Input:Output-Interface-rescue_Output-Interface-rescue_16-way-pcb-edge-Educ-8-connectors-EDUC-8-Input
- R1, R2, R3, R4: symbol Device:R -> Input:Output-Interface-rescue_Output-Interface-rescue_R-Device-Input
Connections:
- wire segments 296 -> 292
Other:
- note added: "00"
- note added: "01"
- note added: "10"
- note added: "11"
- note added: "606"
- note added: "616"
- note added: "626"
- note added: "636"
- note added: "DATA"
- note added: "c"
- moved on the sheet: U2B
Changed lines of the file:
@@
 U 3 1 60BF98A8
 P 7900 2150
-F 0 "U3" H 7900 2150 50  0000 C CNN
-F 1 "7400" H 7900 2350 50  0000 C CNN
+F 0 "U3" H 7900 1850 50  0000 C CNN
+F 1 "7400" H 7900 1950 50  0000 C CNN
 F 2 "" H 7900 2150 50  0001 C CNN
 F 3 "http://www.ti.com/lit/gpn/sn7400" H 7900 2150 50  0001 C CNN
@@
 U 4 1 60BFC749
 P 7900 2750
-F 0 "U3" H 7850 2750 50  0000 C CNN
-F 1 "7400" H 7900 2524 50  0000 C CNN
+F 0 "U3" H 7900 2550 50  0000 C CNN
+F 1 "7400" H 7900 2450 50  0000 C CNN
 F 2 "" H 7900 2750 50  0001 C CNN
 F 3 "http://www.ti.com/lit/gpn/sn7400" H 7900 2750 50  0001 C CNN
 	4    7900 2750
-	-1   0    0    1
+	-1   0    0    -1
 $EndComp
 $Comp
 L 74xx:74LS04 U2
 U 2 1 60C00E16
-P 9450 2250
-F 0 "U2" H 9450 1933 50  0000 C CNN
-F 1 "74LS04" H 9450 2024 50  0000 C CNN
-F 2 "Package_DIP:DIP-14_W7.62mm" H 9450 2250 50  0001 C CNN
-F 3 "http://www.ti.com/lit/gpn/sn74LS04" H 9450 2250 50  0001 C CNN
-	2    9450 2250
-	-1   0    0    1
-$EndComp
-Wire Wire Line
-	9150 800  8400 800
-Wire Wire Line
-	8200 1400 8400 1400
-Wire Wire Line
-	8400 1400 8400 800
-Connection ~ 8400 800
-Wire Wire Line
-	8400 800  8200 800
-Wire Wire Line
-	9750 800  10000 800
-Wire Wire Line
-	8950 2050 8950 1350
-Wire Wire Line
-	8950 1350 10000 1350
-Wire Wire Line
-	10000 1350 10000 800
-Connection ~ 10000 800
-Wire Wire Line
-	10000 800  10550 800
-Wire Wire Line
-	8200 2850 8400 2850
-Wire Wire Line
-	8200 1600 8400 1600
-Wire Wire Line
-	8400 1600 8400 2850
+P 9450 2650
+F 0 "U2" H 9450 2333 50  0000 C CNN
+F 1 "74LS04" H 9450 2424 50  0000 C CNN
+F 2 "Package_DIP:DIP-14_W7.62mm" H 9450 2650 50  0001 C CNN
+F 3 "http://www.ti.com/lit/gpn/sn74LS04" H 9450 2650 50  0001 C CNN
+	2    9450 2650
+	-1   0    0    1
+$EndComp
 Text Label 10250 800  0    50   ~ 0
 6
-Text Label 10250 2250 0    50   ~ 0
+Text Label 10250 2650 0    50   ~ 0
 5
-Wire Wire Line
-	8950 2650 8950 2050
-Connection ~ 8950 2050
-Wire Wire Line
-	8200 2650 8950 2650
-Wire Wire Line
-	8200 2050 8950 2050
 Text GLabel 10550 800  2    50   Input ~ 0
 I_O_GATING
-Text GLabel 10450 2250 2    50   Input ~ 0
+Text GLabel 10450 2650 2    50   Input ~ 0
 I_O_DEVICE_SELECT
 Text Notes 10600 1050 0    50   ~ 0
@@
 	7150 2750 7600 2750
 $Comp
-L Device:R R1
+L Input:Output-Interface-rescue_Output-Interface-rescue_R-Device-Input R1
 U 1 1 60C518AD
 P 7200 8450
@@
 	10500 6800 10500 6900
 $Comp
-L Device:R R4
+L Input:Output-Interface-rescue_Output-Interface-rescue_R-Device-Input R4
 U 1 1 60CF8C83
 P 10150 6900
@@
 $EndComp
 $Comp
-L power:+5V #PWR0101
+L Input:Output-Interface-rescue_Output-Interface-rescue_+5V-power-Input #PWR0101
 U 1 1 60D03E50
 P 9850 6850
@@
 $EndComp
 $Comp
-L Device:R R3
+L Input:Output-Interface-rescue_Output-Interface-rescue_R-Device-Input R3
 U 1 1 60D2FE21
 P 9850 8350
@@
 $EndComp
 $Comp
-L Device:R R2
+L Input:Output-Interface-rescue_Output-Interface-rescue_R-Device-Input R2
 U 1 1 60D30AFF
 P 8550 8350
@@
 	9850 8200 9850 8100
 $Comp
-L power:+5V #PWR0102
+L Input:Output-Interface-rescue_Output-Interface-rescue_+5V-power-Input #PWR0102
 U 1 1 60D3E150
 P 9850 8100
@@
 	8550 8700 9050 8700
 $Comp
-L power:+5V #PWR0103
+L Input:Output-Interface-rescue_Output-Interface-rescue_+5V-power-Input #PWR0103
 U 1 1 60D55945
 P 8550 8100
@@
 	7450 8700 7450 8800
 $Comp
-L power:+5V #PWR0104
+L Input:Output-Interface-rescue_Output-Interface-rescue_+5V-power-Input #PWR0104
 U 1 1 60D9B825
 P 7200 8200
@@
 Connection ~ 7200 8700
 $Comp
-L Connector:Conn_01x03_Male J1
+L Input:Output-Interface-rescue_Output-Interface-rescue_Conn_01x03_Male-Connector-Input J1
 U 1 1 60DB4FBC
 P 7550 6400
@@
 $EndComp
 $Comp
-L Connector:Conn_01x03_Male J2
+L Input:Output-Interface-rescue_Output-Interface-rescue_Conn_01x03_Male-Connector-Input J2
 U 1 1 60DB6847
 P 7550 7000
@@
 	4100 7400 3050 7400
 $Comp
-L EDUC-8:16-way-pcb-edge-Educ-8-connectors J4
+L Input:Output-Interface-rescue_Output-Interface-rescue_16-way-pcb-edge-Educ-8-connectors-EDUC-8-Input J4
 U 1 1 6106ED6B
 P 15350 2350
@@
 T13
 $Comp
-L power:+5V #PWR0105
+L Input:Output-Interface-rescue_Output-Interface-rescue_+5V-power-Input #PWR0105
 U 1 1 61077016
 P 14550 1600
@@
 $EndComp
 $Comp
-L power:GND #PWR0106
+L Input:Output-Interface-rescue_Output-Interface-rescue_GND-power-Input #PWR0106
 U 1 1 61079285
 P 14950 1300
@@
 	14900 2300 15250 2300
 $Comp
-L power:GND #PWR0107
+L Input:Output-Interface-rescue_Output-Interface-rescue_GND-power-Input #PWR0107
 U 1 1 61137FC6
 P 15050 3000
@@
 	15250 3000 15050 3000
 $Comp
-L EDUC-8:16-way-pcb-edge-Educ-8-connectors J3
+L Input:Output-Interface-rescue_Output-Interface-rescue_16-way-pcb-edge-Educ-8-connectors-EDUC-8-Input J3
 U 1 1 611491AA
 P 15350 4400
@@
 Text Notes 10100 750  2    50   ~ 0
 CORRECT
-Text Notes 8550 2050 2    50   ~ 0
+Text Notes 8850 2050 2    50   ~ 0
 CORRECT
-Text Notes 8550 2600 2    50   ~ 0
+Text Notes 8800 2600 2    50   ~ 0
 CORRECT
-Wire Wire Line
-	8200 2250 9100 2250
-Wire Wire Line
-	9850 1000 9850 2250
-Wire Wire Line
-	8200 1000 9850 1000
-Connection ~ 9850 2250
-Wire Wire Line
-	9850 2250 9750 2250
-Wire Wire Line
-	9850 2250 10450 2250
-Wire Wire Line
-	9100 2250 9100 2850
-Wire Wire Line
-	9100 2850 8400 2850
-Connection ~ 9100 2250
-Wire Wire Line
-	9100 2250 9150 2250
-Connection ~ 8400 2850
 Connection ~ 3150 6350
 Connection ~ 3150 5850
@@
 	1850 11000 2850 11000
 $Comp
-L power:+5V #PWR0108
+L Input:Output-Interface-rescue_Output-Interface-rescue_+5V-power-Input #PWR0108
 U 1 1 61A4E904
 P 3100 9750
@@
 $EndComp
 $Comp
-L power:GND #PWR0109
+L Input:Output-Interface-rescue_Output-Interface-rescue_GND-power-Input #PWR0109
 U 1 1 61A507E9
 P 3250 11050
@@
 	5100 5700 5100 7800
 $Comp
-L Device:C C1
+L Input:Output-Interface-rescue_Output-Interface-rescue_C-Device-Input C1
 U 1 1 61D91026
 P 11750 4050
@@
 $EndComp
 $Comp
-L Device:C C2
+L Input:Output-Interface-rescue_Output-Interface-rescue_C-Device-Input C2
 U 1 1 61D91723
 P 12200 4050
@@
 $EndComp
 $Comp
-L Device:C C3
+L Input:Output-Interface-rescue_Output-Interface-rescue_C-Device-Input C3
 U 1 1 61D91989
 P 12650 4050
@@
 $EndComp
 $Comp
-L Device:C C4
+L Input:Output-Interface-rescue_Output-Interface-rescue_C-Device-Input C4
 U 1 1 61D91B02
 P 13100 4050
@@
 	12200 3650 12400 3650
 $Comp
-L power:+5V #PWR0110
+L Input:Output-Interface-rescue_Output-Interface-rescue_+5V-power-Input #PWR0110
 U 1 1 61E2E864
 P 12400 3550
@@
 $EndComp
 $Comp
-L power:GND #PWR0111
+L Input:Output-Interface-rescue_Output-Interface-rescue_GND-power-Input #PWR0111
 U 1 1 61E2EDA5
 P 12450 4500
@@
 	12450 4400 12650 4400
 $Comp
-L EDUC-8:Card_handle H1
+L Input:Output-Interface-rescue_Output-Interface-rescue_Card_handle-EDUC-8-Input H1
 U 1 1 61DFC554
 P 12700 8150
@@
 $EndComp
 $Comp
-L EDUC-8:Card_handle H2
+L Input:Output-Interface-rescue_Output-Interface-rescue_Card_handle-EDUC-8-Input H2
 U 1 1 61DFCEA4
 P 14000 8150
@@
 	1    0    0    -1
 $EndComp
-Wire Wire Line
-	12700 8400 13350 8400
-$Comp
-L power:GND #PWR0112
+$Comp
+L Input:Output-Interface-rescue_Output-Interface-rescue_GND-power-Input #PWR0112
 U 1 1 61E18F0E
 P 13350 8400
@@
 	1    0    0    -1
 $EndComp
-Connection ~ 13350 8400
-Wire Wire Line
-	13350 8400 14000 8400
+Wire Wire Line
+	12700 8400 14000 8400
+Text Notes 7850 1550 0    50   ~ 0
+00
+Text Notes 7850 950  0    50   ~ 0
+01
+Text Notes 7850 2800 0    50   ~ 0
+10
+Text Notes 7850 2200 0    50   ~ 0
+11
+Text Notes 7350 850  0    50   ~ 0
+C
+Text Notes 7400 1450 0    50   ~ 0
+c
+Text Notes 7400 2100 0    50   ~ 0
+c
+Text Notes 7400 2700 0    50   ~ 0
+c
+Text Notes 8250 1350 0    50   ~ 0
+c
+Text Notes 8200 750  0    50   ~ 0
+c
+Wire Wire Line
+	9750 800  10100 800
+Wire Wire Line
+	9750 2650 9950 2650
+Wire Wire Line
+	9150 800  8650 800
+Wire Wire Line
+	8650 1400 8650 800
+Wire Wire Line
+	8200 1400 8650 1400
+Connection ~ 8650 800
+Wire Wire Line
+	8650 800  8200 800
+Wire Wire Line
+	8650 1600 8650 2650
+Wire Wire Line
+	8650 2650 9150 2650
+Wire Wire Line
+	8200 1600 8650 1600
+Wire Wire Line
+	8200 2650 8650 2650
+Connection ~ 8650 2650
+Wire Wire Line
+	8200 1000 9950 1000
+Wire Wire Line
+	9950 1000 9950 2250
+Connection ~ 9950 2650
+Wire Wire Line
+	9950 2650 10450 2650
+Wire Wire Line
+	8200 2250 9950 2250
+Connection ~ 9950 2250
+Wire Wire Line
+	9950 2250 9950 2650
+Wire Wire Line
+	8200 2050 10100 2050
+Wire Wire Line
+	10100 2050 10100 800
+Connection ~ 10100 800
+Wire Wire Line
+	10100 800  10550 800
+Wire Wire Line
+	10100 2050 10100 2850
+Wire Wire Line
+	10100 2850 8200 2850
+Connection ~ 10100 2050
+Text Notes 6150 900  0    50   ~ 0
+616
+Text Notes 6150 1500 0    50   ~ 0
+606
+Text Notes 6150 2150 0    50   ~ 0
+636
+Text Notes 6150 2750 0    50   ~ 0
+626
+Text Notes 6150 3400 0    50   ~ 0
+DATA
 $EndSCHEMATC
