File: Octal display/Octal display.kicad_pcb (KiCad board)
At the start: 2 copper layers, 140 x 100 mm, 74 parts, among them J1 Conn_01x08_Female, J2 Conn_01x04_Female, J3 Conn_01x04_Male, J4 Conn_01x04_Female, Q1 BC547, Q10 BC547, Q11 BC547, Q12 BC547, Q13 BC547, Q14 BC547, Q15 BC547, Q16 BC547, Q17 BC547, Q18 BC547, Q19 BC547, Q2 BC547, Q20 BC547, Q21 BC547, Q23 BC108, Q24 BC108, Q3 BC547, Q4 BC547, Q5 BC547, Q6 BC547, Q7 BC547, Q8 BC547, Q9 BC547, U1 74164, U2 74LS48, U3 74LS48, U4 74LS48, U5 74LS37, U6 74LS13

Commit message: Schematic update 2024-04-14 plus fixes
Parts:
- Q1, Q10, Q11, Q12, Q13, Q14, Q15, Q16, Q17, Q18, Q19, Q2, Q20, Q21, Q3, Q4, Q5, Q6, Q7, Q8, Q9: footprint Package_TO_SOT_THT:TO-92_Inline -> Package_TO_SOT_THT:TO-92_Inline_Wide
- moved Q7 1.70 mm to (82.4, 65.5)
- moved Q12 1.11 mm to (127.2, 85.2)
- moved Q6 0.91 mm to (75.4, 66.2)
- moved Q5 0.86 mm to (82.1, 85.2)
- moved Q3 0.85 mm to (72.0, 85.2)
- moved Q17 0.85 mm to (163.0, 85.2)
- moved Q1 0.85 mm to (62.0, 85.2)
- moved Q10 0.85 mm to (117.0, 85.2)
- moved Q11 0.85 mm to (122.0, 85.2)
- moved Q13 0.85 mm to (97.0, 85.2)
- moved Q14 0.85 mm to (102.0, 85.2)
- moved Q15 0.85 mm to (153.0, 85.2)
- moved Q16 0.85 mm to (158.0, 85.2)
- moved Q18 0.85 mm to (168.0, 85.2)
- moved Q19 0.85 mm to (173.0, 85.2)
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Routing:
- net Net-(Q7-Pad2): track 61.1 -> 63.9 mm
- net Net-(AFF2-Pad9): track 39.3 -> 37.0 mm
- net Net-(Q2-Pad2): track 24.8 -> 26.7 mm
- net Net-(Q7-Pad1): track 13.1 -> 14.9 mm
- net Net-(Q10-Pad2): track 23.8 -> 25.5 mm
- net Net-(Q16-Pad2): track 24.5 -> 26.0 mm
- net Net-(Q18-Pad2): track 22.4 -> 23.9 mm
- net Net-(Q17-Pad2): track 23.6 -> 25.1 mm
- net Net-(AFF1-Pad10): track 9.33 -> 7.84 mm
- net Net-(Q3-Pad2): track 23.8 -> 25.3 mm
- net Net-(Q20-Pad2): track 27.1 -> 28.5 mm
- net Net-(Q9-Pad2): track 25.5 -> 26.9 mm
- net Net-(Q11-Pad2): track 24.0 -> 25.4 mm
- net Net-(Q19-Pad2): track 26.1 -> 24.9 mm
- net Net-(AFF2-Pad1): track 30.4 -> 29.3 mm
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