File: Octal display/Octal display.kicad_sch (KiCad schematic)
At the start: 73 parts, among them J1 Conn_01x08_Female, J2 Conn_01x04_Female, J3 Conn_01x04_Male, J4 Conn_01x04_Female, Q1 BC547, Q10 BC547, Q11 BC547, Q12 BC547, Q13 BC547, Q14 BC547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

Commit message: Schematic update 2024-04-14 plus fixes
Parts:
- Q1, Q10, Q11, Q12, Q13, Q14, Q15, Q16, Q17, Q18, Q19, Q2, Q20, Q21, Q3, Q4, Q5, Q6, Q7, Q8, Q9: footprint Package_TO_SOT_THT:TO-92_Inline -> Package_TO_SOT_THT:TO-92_Inline_Wide
- U5: footprint (none) -> Package_DIP:DIP-14_W7.62mm
