File: Octal display/Pot and switch board/support PCB/support PCB.kicad_pcb (KiCad board)
At the start: 2 copper layers, 140 x 100 mm, 19 parts, among them J1 Conn_01x04_Male, J2 Conn_01x08_Male, J3 Conn_01x04_Male, J4 Conn_01x04_Male, J5 DIN-6_SH, K1 FRT5, K2 FRT5, K3 FRT5, SW1 SW_DPDT_x2

Commit message: Schematic update 2024-04-14 plus fixes
Connections:
- net ~CLOCK renamed ~{CLOCK}
- net ~DATA renamed ~{DATA}
- net ~FLAG renamed ~{FLAG}
- net ~FLAG_RESET renamed ~{FLAG_RESET}
- net ~RBI renamed ~{RBI}
Other:
- net class Default removed
