File: motherboard/motherboard.sch (KiCad schematic (older format))
At the start: 44 parts, among them J1 E8/T, J10 36-way-edge-connector, J11 36-way-edge-connector, J12 Conn_01x08_Female, J13 Conn_01x08_Female, J14 Conn_01x16_Female, J15 Conn_01x04_Female, J16 Conn_01x04_Female, J17 Conn_01x01_Female, J18 Conn_01x04_Female, J19 Conn_01x08_Female, J2 36-way-pcb-edge-socket-Educ-8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, J20 Conn_01x04_Female, J21 Conn_01x04_Female, J22 Conn_01x04_Female, J23 Conn_01x04_Female, J24 Conn_01x04_Female, J25 Conn_01x04_Female, J26 Conn_01x04_Female, J27 Conn_01x04_Female, J28 Conn_01x04_Female, J29 Conn_01x01_Female, J3 36-way-pcb-edge-socket-Educ-8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, J30 Conn_01x01_Female, J31 Conn_01x01_Female, J4 36-way-pcb-edge-socket-Educ-8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, J5 36-way-edge-connector, J6 36-way-edge-connector, J7 36-way-edge-connector, J8 36-way-edge-connector, J9 36-way-edge-connector

Commit message: Schematic update 2024-04-14 plus fixes
Parts:
- C1, C2, C3: symbol Device:C -> motherboard-rescue:C-Device
- H1, H2, H3, H4, H5, H6: symbol Mechanical:MountingHole_Pad -> motherboard-rescue:MountingHole_Pad-Mechanical
- J12, J13, J19: symbol Connector:Conn_01x08_Female -> motherboard-rescue:Conn_01x08_Female-Connector
- J14: symbol Connector:Conn_01x16_Female -> motherboard-rescue:Conn_01x16_Female-Connector
- J15, J16, J18, J20, J21, J22, J23, J24, J25, J26, J27, J28: symbol Connector:Conn_01x04_Female -> motherboard-rescue:Conn_01x04_Female-Connector
- J17, J29, J30, J31: symbol Connector:Conn_01x01_Female -> motherboard-rescue:Conn_01x01_Female-Connector
- R1, R2, R3, R4: symbol Device:R -> motherboard-rescue:R-Device
