File: motherboard/motherboard.kicad_pcb (KiCad board)
At the start: 2 copper layers, 283 x 96 mm, 47 parts, among them J1 E8/T, J10 36-way-edge-connector, J11 36-way-edge-connector, J12 Conn_01x08_Female, J13 Conn_01x08_Female, J14 Conn_01x16_Female, J15 Conn_01x04_Female, J16 Conn_01x04_Female, J17 Conn_01x02_Female, J18 Conn_01x04_Female, J19 Conn_01x08_Female, J2 36-way-pcb-edge-socket-Educ-8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, J20 Conn_01x04_Female, J21 Conn_01x04_Female, J22 Conn_01x04_Female, J23 Conn_01x04_Female, J24 Conn_01x04_Female, J25 Conn_01x04_Female, J26 Conn_01x04_Female, J27 Conn_01x04_Female, J28 Conn_01x04_Female, J29 Conn_01x02_Female, J3 36-way-pcb-edge-socket-Educ-8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, J30 Conn_01x01_Female, J31 Conn_01x01_Female, J32 TO_E8/M, J33 TO_E8/P, J4 36-way-pcb-edge-socket-Educ-8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, J5 36-way-edge-connector, J6 36-way-edge-connector, J7 36-way-edge-connector, J8 36-way-edge-connector, J9 36-way-edge-connector

Commit message: Schematic update 2024-04-14 plus fixes
Parts:
- added J34: Conn_01x05_Male, Connector_JST:JST_XH_B5B-XH-AM_1x05_P2.50mm_Vertical, F.Cu at (269.5, 245.5)
- added J35: Conn_01x05_Male, Connector_JST:JST_XH_B5B-XH-AM_1x05_P2.50mm_Vertical, F.Cu at (287.6, 245.4)
- added J36: Conn_01x02_Male, Connector_JST:JST_XH_B2B-XH-AM_1x02_P2.50mm_Vertical, F.Cu at (37.0, 186.0)
- J25: value Conn_01x04_Female -> Conn_01x03_Male; footprint Connector_Molex:Molex_KK-254_AE-6410-04A_1x04_P2.54mm_Vertical -> Connector_JST:JST_XH_B3B-XH-AM_1x03_P2.50mm_Vertical
- J26: value Conn_01x04_Female -> Conn_01x10_Female; footprint Connector_Molex:Molex_KK-254_AE-6410-04A_1x04_P2.54mm_Vertical -> Connector_JST:JST_XH_B10B-XH-AM_1x10_P2.50mm_Vertical
- J27, J28: value Conn_01x04_Female -> Conn_01x05_Male; footprint Connector_Molex:Molex_KK-254_AE-6410-04A_1x04_P2.54mm_Vertical -> Connector_JST:JST_XH_B5B-XH-AM_1x05_P2.50mm_Vertical
- R4: value R -> 680R
- moved J29 116.1 mm to (295.9, 158.4), turned to 90 degrees
- moved J26 49.8 mm to (198.9, 239.2)
- moved J25 44.0 mm to (186.8, 239.2)
- moved J27 41.4 mm to (228.0, 245.6)
- moved J28 41.4 mm to (246.0, 245.5)
Connections:
- net Net-(J14-Pad11) renamed /MA5
- net Net-(J14-Pad12) renamed /MA6
- net Net-(J14-Pad13) renamed /MA7
- J1 pad A1: (no net) -> unconnected-(J1-PadA1)
- J1 pad A10: (no net) -> ~{DEP+EXM}
- J1 pad A11: (no net) -> FAST_SLOW
- J1 pad A12: (no net) -> ~{T0.5}
- J1 pad A13: (no net) -> ~{T0+T12}
- J1 pad A14: (no net) -> T14-21
- J1 pad A15: (no net) -> MCPB
- J1 pad A16: (no net) -> T14-21
- J1 pad A17: (no net) -> MCPA
- J1 pad A18: (no net) -> T13
- J1 pad A19: (no net) -> T2-9
- J1 pad A2: (no net) -> unconnected-(J1-PadA2)
- J1 pad A20: (no net) -> T1
- J1 pad A21: (no net) -> ~{CANCEL+DEP+EXM}
- J1 pad A22: (no net) -> ~{F.T23.}OPR+IOT
- J1 pad A23: (no net) -> F.2-9(F+D+E)
- J1 pad A24: (no net) -> OPR+IOT
- J1 pad A25: (no net) -> FETCH
- J1 pad A26: (no net) -> unconnected-(J1-PadA26)
- J1 pad A27: (no net) -> EXECUTE
- J1 pad A28: (no net) -> ~{F+D+E}
- J1 pad A29: (no net) -> unconnected-(J1-PadA29)
- J1 pad A3: (no net) -> unconnected-(J1-PadA3)
- J1 pad A30: (no net) -> unconnected-(J1-PadA30)
- J1 pad A31: (no net) -> ~{RUN}
- J1 pad A32: (no net) -> ~{FETCH}
- J1 pad A33: (no net) -> ~{DEFER}
- J1 pad A34: (no net) -> ~{EXEC}
- J1 pad A35: (no net) -> MB4
- J1 pad A36: (no net) -> GND
- J1 pad A4: (no net) -> unconnected-(J1-PadA4)
- J1 pad A5: (no net) -> GND
- J1 pad A6: (no net) -> +5V
- J1 pad A7: (no net) -> T22.5
- J1 pad A8: (no net) -> ~{RUN_COMMAND}
- J1 pad A9: (no net) -> HALT_COMMAND
- J1 pad H1: (no net) -> GND
- J1 pad H2: (no net) -> GND
- J2 pad A1: (no net) -> unconnected-(J2-PadA1)
- J2 pad A10: (no net) -> ~{CLEAR_IOT_FLAG}
- J2 pad A11: (no net) -> SKP_ON_IOT_FLAG
- J2 pad A12: (no net) -> ~{T0.5}
- J2 pad A13: (no net) -> T14-21
- J2 pad A14: (no net) -> T14-21
- J2 pad A15: (no net) -> ~{IOT_SHIFT}
- J2 pad A16: (no net) -> T2-9
- J2 pad A17: (no net) -> ~{T2-9.(TAD+IAC+CMA})
- J2 pad A18: (no net) -> T2-9.ISZ
- J2 pad A19: (no net) -> JMS+DCA
- J2 pad A2: (no net) -> unconnected-(J2-PadA2)
- J2 pad A20: (no net) -> OPR+IOT
- J2 pad A21: (no net) -> ~{T14-21(JMS+JMP})
- J2 pad A22: (no net) -> ~{T14-21.SKP}
- J2 pad A23: (no net) -> FETCH
- J2 pad A24: (no net) -> ~{DEFER}
- J2 pad A25: (no net) -> EXECUTE
- J2 pad A26: (no net) -> ~{F+D+E}
- J2 pad A27: (no net) -> MEM.ENABLE
- J2 pad A28: (no net) -> ~{HLT}
- J2 pad A29: (no net) -> ~{RAR}
- J2 pad A3: (no net) -> unconnected-(J2-PadA3)
- J2 pad A30: (no net) -> ~{SMA}
- J2 pad A31: (no net) -> ~{SZA}
- J2 pad A32: (no net) -> ~{IAC}
- J2 pad A33: (no net) -> ~{RAL}
- J2 pad A34: (no net) -> ~{CMA}
- J2 pad A35: (no net) -> ~{CLA}
- J2 pad A36: (no net) -> GND
- J2 pad A4: (no net) -> unconnected-(J2-PadA4)
- J2 pad A5: (no net) -> GND
- J2 pad A6: (no net) -> +5V
- J2 pad A7: (no net) -> T22.5
- J2 pad A8: (no net) -> IO_DEVICE_SELECT
- J2 pad A9: (no net) -> IO_GATING
- J2 pad H1: (no net) -> GND
- J2 pad H2: (no net) -> GND
- J25 pad 1: OD1_~{DATA} -> SR5
- J25 pad 2: OD1~{FLAG} -> SR6
- J25 pad 3: OD1~{FLAG_RESET} -> SR7
- J26 pad 1: OD0~{DATA} -> GND
- J26 pad 2: OD0~{FLAG} -> SR0
- J26 pad 3: OD0~{FLAG_RESET} -> SR1
- J26 pad 4: OD0~{CLK} -> SR2
- J27 pad 1: ID1~{DATA} -> GND
- J27 pad 2: ID1~{FLAG} -> OD1_~{DATA}
- J27 pad 3: ID1~{FLAG_RESET} -> OD1~{FLAG}
- J27 pad 4: ID1~{CLK} -> OD1~{FLAG_RESET}
- J28 pad 1: ID0~{DATA} -> GND
- J28 pad 2: ID0~{FLAG} -> OD0~{DATA}
- J28 pad 3: ID0~{FLAG_RESET} -> OD0~{FLAG}
- J28 pad 4: ID0~{CLK} -> OD0~{FLAG_RESET}
- J3 pad A1: (no net) -> unconnected-(J3-PadA1)
- J3 pad A10: (no net) -> D-BUS
- J3 pad A11: (no net) -> ~{T0.5}
- J3 pad A12: (no net) -> T14-21
- J3 pad A13: (no net) -> MCPB
- J3 pad A14: (no net) -> T13
- J3 pad A15: (no net) -> T2-9
- J3 pad A16: (no net) -> T1
- J3 pad A17: (no net) -> T2-9.ISZ
- J3 pad A18: (no net) -> ~{F.T23.}OPR+IOT
- J3 pad A19: (no net) -> F.2-9(F+D+E)
- J3 pad A2: (no net) -> unconnected-(J3-PadA2)
- J3 pad A20: (no net) -> OPR+IOT
- J3 pad A21: (no net) -> ~{T14-21(JMS+JMP})
- J3 pad A22: (no net) -> JMS+DCA
- J3 pad A23: (no net) -> ~{DEP}
- J3 pad A24: (no net) -> unconnected-(J3-PadA24)
- J3 pad A25: (no net) -> unconnected-(J3-PadA25)
- J3 pad A26: (no net) -> ~{F+D+E}
- J3 pad A27: (no net) -> MEM.ENABLE
- J3 pad A28: (no net) -> SR0
- J3 pad A29: (no net) -> SR1
- J3 pad A3: (no net) -> unconnected-(J3-PadA3)
- J3 pad A30: (no net) -> SR2
- J3 pad A31: (no net) -> SR3
- J3 pad A32: (no net) -> SR4
- J3 pad A33: (no net) -> SR5
- J3 pad A34: (no net) -> SR6
- J3 pad A35: (no net) -> SR7
- J3 pad A36: (no net) -> GND
- J3 pad A4: (no net) -> unconnected-(J3-PadA4)
- J3 pad A5: (no net) -> GND
- J3 pad A6: (no net) -> +5V
- J3 pad A7: (no net) -> +5V
- J3 pad A8: (no net) -> B-BUS
- J3 pad A9: (no net) -> C-BUS
- J3 pad H1: (no net) -> GND
- J3 pad H2: (no net) -> GND
- J4 pad A1: (no net) -> unconnected-(J4-PadA1)
- J4 pad A10: (no net) -> C-BUS
- J4 pad A11: (no net) -> D-BUS
- J4 pad A12: (no net) -> ~{T0+T12}
- J4 pad A13: (no net) -> ~{T13.RAR}
- J4 pad A14: (no net) -> ~{IOT_SKP}
- J4 pad A15: (no net) -> MCPA
- J4 pad A16: (no net) -> T13
- J4 pad A17: (no net) -> T2-9
- J4 pad A18: (no net) -> T1
- J4 pad A19: (no net) -> ~{T2-9.(TAD+IAC+CMA})
- J4 pad A2: (no net) -> unconnected-(J4-PadA2)
- J4 pad A20: (no net) -> AC=0
- J4 pad A21: (no net) -> ~{LA1}
- J4 pad A22: (no net) -> LA2
- J4 pad A23: (no net) -> T2-9.ISZ
- J4 pad A24: (no net) -> F.2-9(F+D+E)
- J4 pad A25: (no net) -> ~{T14-21(JMS+JMP})
- J4 pad A26: (no net) -> ~{T14-21.SKP}
- J4 pad A27: (no net) -> ~{F+D+E}
- J4 pad A28: (no net) -> SR0
- J4 pad A29: (no net) -> SR1
- J4 pad A3: (no net) -> unconnected-(J4-PadA3)
- J4 pad A30: (no net) -> SR2
- J4 pad A31: (no net) -> SR3
- J4 pad A32: (no net) -> SR4
- J4 pad A33: (no net) -> SR5
- J4 pad A34: (no net) -> ~{SMA}
- J4 pad A35: (no net) -> ~{SZA}
- J4 pad A36: (no net) -> GND
- J4 pad A4: (no net) -> unconnected-(J4-PadA4)
- J4 pad A5: (no net) -> GND
- J4 pad A6: (no net) -> +5V
- J4 pad A7: (no net) -> +5V
- J4 pad A8: (no net) -> A-BUS
- J4 pad A9: (no net) -> B-BUS
- J4 pad H1: (no net) -> GND
- J4 pad H2: (no net) -> GND
Routing:
- net HALT_COMMAND: track 3.96 -> 126.8 mm
- net GND: track 400.1 -> 284.1 mm, vias 8 -> 9
- net +5V: track 142.3 -> 254.3 mm
- net Z-BIT: track 3.96 -> 110.0 mm
- net ~{EXT.LA}: track 2.54 -> 75.2 mm
- net AC=0: track 50.9 -> 16.1 mm
- net SR7: track 65.7 -> 98.5 mm
- net SR6: track 64.7 -> 96.9 mm
- net SR5: track 73.7 -> 105.1 mm
- net ~{EXT.DEP}: track 0.00 -> 15.1 mm
- net AC0_TO_IOT: track 3.96 -> 16.1 mm
- net ~{RUN_COMMAND}: track 63.4 -> 54.0 mm
- net ~{HLT}: track 198.6 -> 194.1 mm
- net ~{CMA}: track 139.0 -> 135.5 mm
- net ~{DEP}: track 255.2 -> 252.1 mm
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Other:
- board text added: "TO E8/P"

Commit message: Changes 20-7-2025 E8/T. Connected 3 missing supply rail tracks to ICS Added flood fill top and bottom to reduce noise E8/F Corrected labelling on RHS board to reflect EXT_LA not GND Changed fast slow switch operation so fast is in the DOWN position. E8/C. Ran a new track to the 2 pin JST connector from EXT_LA from 10 pin connector on SR input. Added files for E8MX, 2k byte memory expansion board
Parts:
- added J37: Conn_01x02_Male, Connector_JST:JST_XH_B2B-XH-A_1x02_P2.50mm_Vertical, F.Cu at (262.9, 238.9)
- J1: value E8/T -> E8/T
- J17: moved to B.Cu
- J25: value Conn_01x03_Male -> TO E8/P
- J29: value Conn_01x02_Female -> Conn_01x02_Male; footprint Connector_PinSocket_2.54mm:PinSocket_1x02_P2.54mm_Vertical -> Connector_JST:JST_XH_B2B-XH-AM_1x02_P2.50mm_Vertical
- moved J29 0.22 mm to (296.1, 158.4), turned to 0 degrees
- turned J17 to 90 degrees
Connections:
- J1 pad 14: T14-21 -> T14-21A
- J1 pad A14: T14-21 -> T14-21A
- J2 pad 13: T14-21 -> T14-21A
- J2 pad A13: T14-21 -> T14-21A
- J23 pad 3: GND -> unconnected-(J23-Pin_3-Pad3)
- J26 pad 10: ~{EXT.LA} -> Net-(J26-Pin_10)
- J3 pad 12: T14-21 -> T14-21A
- J3 pad A12: T14-21 -> T14-21A
- J36 pad 1: GND -> ~{EXT.LA}
- J9 pad 8: AC=-VE -> AC7
- J9 pad H: AC=-VE -> AC7
Routing:
- net ~{EXT.LA}: track 75.2 -> 307.8 mm
- net AC7: track 36.1 -> 74.8 mm
- net T14-21: track 48.6 -> 20.3 mm
- net T14-21A: track 0.00 -> 28.2 mm
- net AC=-VE: track 3.96 -> 0.00 mm
- net GND: track 284.1 -> 280.7 mm
- net ID1~{FLAG}: track 32.0 -> 29.0 mm
- net ID1~{FLAG_RESET}: track 29.5 -> 27.4 mm
- net ID1~{DATA}: track 32.9 -> 31.7 mm
- net T2-9: track 76.0 -> 77.0 mm
- net ID1~{CLK}: track 27.9 -> 27.1 mm
Other:
- board text added: "50 YEARS"
- board text added: "Designed by Jamieson Rowe 1974 Electroncis Australia PCB by Gwyllym Suter 2024 Special thanks to Steven Pietrobon"
- board text added: "EXT LA"
- board text added: "PAGE ZERO"
- board text added: "SR5-7"
- board text added: "~{EXT.DEP}"
- board text removed: "Designed by Jamieson Rowe 1974 Electroncis Australia PCB by Gwyllym Suter 2021"
- board text removed: "~{EXT. DEP }"
