File: motherboard/motherboard.kicad_sch (KiCad schematic)
At the start: 46 parts, among them J1 E8/T, J10 36-way-edge-connector, J11 36-way-edge-connector, J12 Conn_01x08_Female, J13 Conn_01x08_Female, J14 Conn_01x16_Female, J15 Conn_01x04_Female, J16 Conn_01x04_Female, J18 Conn_01x04_Female, J19 Conn_01x08_Female, J2 36-way-pcb-edge-socket-Educ-8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, J20 Conn_01x04_Female, J21 Conn_01x04_Female, J22 Conn_01x04_Female, J23 Conn_01x04_Female, J24 Conn_01x04_Female, J25 Conn_01x04_Female, J26 Conn_01x04_Female, J27 Conn_01x04_Female, J28 Conn_01x04_Female, J29 Conn_01x02_Female, J3 36-way-pcb-edge-socket-Educ-8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, J30 Conn_01x01_Female, J31 Conn_01x01_Female, J5 36-way-edge-connector, J6 36-way-edge-connector, J7 36-way-edge-connector, J8 36-way-edge-connector, J9 36-way-edge-connector

Commit message: Schematic update 2024-04-14 plus fixes
Parts:
- removed J25, J26, J27, J28: Conn_01x04_Female, Connector_Molex:Molex_KK-254_AE-6410-04A_1x04_P2.54mm_Vertical, symbol Connector:Conn_01x04_Female
- added J25: Conn_01x03_Male, symbol Connector:Conn_01x03_Male
- added J26: Conn_01x10_Female, Connector_JST:JST_XH_B10B-XH-AM_1x10_P2.50mm_Vertical, symbol Connector:Conn_01x10_Female
- added J27, J28, J34, J35: Conn_01x05_Male, Connector_JST:JST_XH_B5B-XH-AM_1x05_P2.50mm_Vertical, symbol Connector:Conn_01x05_Male
- added J36: Conn_01x02_Male, Connector_JST:JST_XH_B2B-XH-AM_1x02_P2.50mm_Vertical, symbol Connector:Conn_01x02_Male
- J1, J2, J3: symbol EDUC8:72-way-edge-connector-Educ-8-connectors -> EDUC8:72-way-edge-connector-Educ-8-connectors_1
- J17: value (none) -> Conn_01x02_Female; footprint (none) -> Connector_PinSocket_2.54mm:PinSocket_1x02_P2.54mm_Vertical
- J32: value (none) -> TO_E8/M
- J33: value (none) -> TO_E8/P; footprint (none) -> Connector_JST:JST_XA_B03B-XASK-1_1x03_P2.50mm_Vertical
- J4: value (none) -> 36-way-pcb-edge-socket-Educ-8-connectors; footprint (none) -> Connector_PCBEdge:72_way_3.96mm_card_edge_socket; symbol EDUC8:72-way-edge-connector-Educ-8-connectors -> EDUC8:72-way-edge-connector-Educ-8-connectors_1
- R4: value (none) -> 680R
Connections:
- net +5V: now also J1.A6, J2.A6, J3.A6, J3.A7, J4.A6, J4.A7; no longer J1.F, J2.F, J3.F, J3.G, J4.F, J4.G
- net A-BUS: now also J4.A8; no longer J4.H
- net AC=0: now also J4.A20; no longer J4.W
- net B-BUS: now also J3.A8, J4.A9; no longer J3.H, J4.J
- net C-BUS: now also J3.A9, J4.A10; no longer J3.J, J4.K
- net D-BUS: now also J3.A10, J4.A11; no longer J3.K, J4.L
- net EXECUTE: now also J1.A27, J2.A25; no longer J1.AD, J2.AB
- net F.2-9(F+D+E): now also J1.A23, J3.A19, J4.A24; no longer J1.Z, J3.V, J4.AA
- net FAST_SLOW: now also J1.A11; no longer J1.L
- net FETCH: now also J1.A25, J2.A23; no longer J1.AB, J2.Z
- net GND: now also J1.A36, J1.A5, J1.H1 (GND), J1.H2 (GND), J2.A36, J2.A5, J2.H1 (GND), J2.H2 (GND), J3.A36, J3.A5, J3.H1 (GND), J3.H2 (GND), J4.A36, J4.A5, J4.H1 (GND), J4.H2 (GND), J26.1 (Pin_1), J27.1 (Pin_1), J28.1 (Pin_1), J34.1 (Pin_1), J35.1 (Pin_1), J36.1 (Pin_1); no longer J1.0 (GND), J1.AN, J1.E, J2.0 (GND), J2.AN, J2.E, J3.0 (GND), J3.AN, J3.E, J4.0 (GND), J4.AN, J4.E
- net HALT_COMMAND: now also J1.A9; no longer J1.J
- net ID0~{CLK}: now also J35.5 (Pin_5)
- net ID0~{DATA}: now also J35.2 (Pin_2)
- net ID0~{FLAG_RESET}: now also J35.4 (Pin_4)
- net ID0~{FLAG}: now also J35.3 (Pin_3)
- net ID1~{CLK}: now also J34.5 (Pin_5)
- net ID1~{DATA}: now also J34.2 (Pin_2)
- net ID1~{FLAG_RESET}: now also J34.4 (Pin_4)
- net ID1~{FLAG}: now also J34.3 (Pin_3)
- net IO_DEVICE_SELECT: now also J2.A8; no longer J2.H
- net IO_GATING: now also J2.A9; no longer J2.J
- net JMS+DCA: now also J2.A19, J3.A22; no longer J2.V, J3.Y
- net LA2: now also J4.A22; no longer J4.Y
- net MB4: now also J1.A35; no longer J1.AM
- net MCPA: now also J1.A17, J4.A15; no longer J1.T, J4.R
- net MCPB: now also J1.A15, J3.A13; no longer J1.R, J3.N
- net MEM.ENABLE: now also J2.A27, J3.A27; no longer J2.AD, J3.AD
- net OD0~{CLK}: now also J28.5 (Pin_5)
- net OD0~{DATA}: now also J28.2 (Pin_2)
- net OD0~{FLAG_RESET}: now also J28.4 (Pin_4)
- net OD0~{FLAG}: now also J28.3 (Pin_3)
- net OD1_~{DATA}: now also J27.2 (Pin_2)
- net OD1~{CLK}: now also J27.5 (Pin_5)
- net OD1~{FLAG_RESET}: now also J27.4 (Pin_4)
- net OD1~{FLAG}: now also J27.3 (Pin_3)
- net OPR+IOT: now also J1.A24, J2.A20, J3.A20; no longer J1.AA, J2.W, J3.W
- net SKP_ON_IOT_FLAG: now also J2.A11; no longer J2.L
- net SR0: now also J3.A28, J4.A28, J26.2 (Pin_2); no longer J3.AE, J4.AE
- net SR1: now also J3.A29, J4.A29, J26.3 (Pin_3); no longer J3.AF, J4.AF
- net SR2: now also J3.A30, J4.A30, J26.4 (Pin_4); no longer J3.AG, J4.AG
- net SR3: now also J3.A31, J4.A31, J26.5 (Pin_5); no longer J3.AH, J4.AH
- net SR4: now also J3.A32, J4.A32, J26.6 (Pin_6); no longer J3.AJ, J4.AJ
- net SR5: now also J3.A33, J4.A33, J25.1 (Pin_1), J26.7 (Pin_7); no longer J3.AK, J4.AK
- net SR6: now also J3.A34, J25.2 (Pin_2), J26.8 (Pin_8); no longer J3.AL
- net SR7: now also J3.A35, J25.3 (Pin_3), J26.9 (Pin_9); no longer J3.AM
- net T1: now also J1.A20, J3.A16, J4.A18; no longer J1.W, J3.S, J4.U
- net T13: now also J1.A18, J3.A14, J4.A16; no longer J1.U, J3.P, J4.S
- net T14-21: now also J1.A14, J1.A16, J2.A13, J2.A14, J3.A12; no longer J1.P, J1.S, J2.N, J2.P, J3.M
- net T2-9: now also J1.A19, J2.A16, J3.A15, J4.A17; no longer J1.V, J2.S, J3.R, J4.T
- net T2-9.ISZ: now also J2.A18, J3.A17, J4.A23; no longer J2.U, J3.T, J4.Z
- net T22.5: now also J1.A7, J2.A7; no longer J1.G, J2.G
- net ~{CANCEL+DEP+EXM}: now also J1.A21; no longer J1.X
- net ~{CLA}: now also J2.A35; no longer J2.AM
- net ~{CLEAR_IOT_FLAG}: now also J2.A10; no longer J2.K
- net ~{CMA}: now also J2.A34; no longer J2.AL
- net ~{DEFER}: now also J1.A33, J2.A24; no longer J1.AK, J2.AA
- net ~{DEP+EXM}: now also J1.A10; no longer J1.K
- net ~{DEP}: now also J3.A23; no longer J3.Z
- net ~{EXEC}: now also J1.A34; no longer J1.AL
- net ~{EXT.DEP}: now also J36.2 (Pin_2)
- net ~{EXT.LA}: now also J26.10 (Pin_10)
- net ~{F+D+E}: now also J1.A28, J2.A26, J3.A26, J4.A27; no longer J1.AE, J2.AC, J3.AC, J4.AD
- net ~{F.T23.}OPR+IOT: now also J1.A22, J3.A18; no longer J1.Y, J3.U
- net ~{FETCH}: now also J1.A32; no longer J1.AJ
- net ~{HLT}: now also J2.A28; no longer J2.AE
- net ~{IAC}: now also J2.A32; no longer J2.AJ
- net ~{IOT_SHIFT}: now also J2.A15; no longer J2.R
- net ~{IOT_SKP}: now also J4.A14; no longer J4.P
- net ~{LA1}: now also J4.A21; no longer J4.X
- net ~{RAL}: now also J2.A33; no longer J2.AK
- net ~{RAR}: now also J2.A29; no longer J2.AF
- net ~{RUN_COMMAND}: now also J1.A8; no longer J1.H
- net ~{RUN}: now also J1.A31; no longer J1.AH
- net ~{SMA}: now also J2.A30, J4.A34; no longer J2.AG, J4.AL
- net ~{SZA}: now also J2.A31, J4.A35; no longer J2.AH, J4.AM
- net ~{T0+T12}: now also J1.A13, J4.A12; no longer J1.N, J4.M
- net ~{T0.5}: now also J1.A12, J2.A12, J3.A11; no longer J1.M, J2.M, J3.L
- net ~{T13.RAR}: now also J4.A13; no longer J4.N
- net ~{T14-21(JMS+JMP}): now also J2.A21, J3.A21, J4.A25; no longer J2.X, J3.X, J4.AB
- net ~{T14-21.SKP}: now also J2.A22, J4.A26; no longer J2.Y, J4.AC
- net ~{T2-9.(TAD+IAC+CMA}): now also J2.A17, J4.A19; no longer J2.T, J4.V
- no-connect marks 65 -> 67
Other:
- moved on the sheet: J17

Commit message: Changes 20-7-2025 E8/T. Connected 3 missing supply rail tracks to ICS Added flood fill top and bottom to reduce noise E8/F Corrected labelling on RHS board to reflect EXT_LA not GND Changed fast slow switch operation so fast is in the DOWN position. E8/C. Ran a new track to the 2 pin JST connector from EXT_LA from 10 pin connector on SR input. Added files for E8MX, 2k byte memory expansion board
Parts:
- removed J29: Conn_01x02_Female, Connector_PinSocket_2.54mm:PinSocket_1x02_P2.54mm_Vertical, symbol Connector:Conn_01x02_Female
- added J29, J37: Conn_01x02_Male, Connector_JST:JST_XH_B2B-XH-AM_1x02_P2.50mm_Vertical, symbol Connector:Conn_01x02_Male
- J1: value E8/T -> E8/T
- J17: now not fitted
- J25: value Conn_01x03_Male -> TO E8/P
Connections:
- net AC=-VE is gone; now on net AC7: J9.8, J9.H
- net GND: now also J7.0 (GND), J37.1 (Pin_1); no longer J23.3 (Pin_3), J36.1 (Pin_1)
- net T14-21: no longer J1.14, J1.A14, J2.13, J2.A13, J3.12, J3.A12
- net Z-BIT: now also J29.1 (Pin_1), J29.2 (Pin_2)
- net ~{EXT.LA}: now also J36.1 (Pin_1); no longer J17.1 (Pin_1), J17.2 (Pin_2), J26.10 (Pin_10)
- new net: J17.1 (Pin_1), J17.2 (Pin_2), J26.10 (Pin_10), J37.2 (Pin_2)
- new net T14-21A: J1.14, J1.A14, J2.13, J2.A13, J3.12, J3.A12
- no-connect marks 67 -> 70
Other:
- note added: "ADD LINK"
- note added: "CUT"
- note added: "MODIFICATION TO MOTHERBARD PRIOR TO 2ND JUNE 2024"
- note added: "See Steven Pietrobon's paper on LS series resistor modifications"
- note added: "THIS SECTION IS REDUNDANT"
- moved on the sheet: C1, C2, C3, J12, J13, J14, J15, J16, J18, J19, J20, J21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
