File: 256 word memory/256 word memory 3.kicad_sch (KiCad schematic)
At the start: 36 parts

Commit message: Changes 20-7-2025 E8/T. Connected 3 missing supply rail tracks to ICS Added flood fill top and bottom to reduce noise E8/F Corrected labelling on RHS board to reflect EXT_LA not GND Changed fast slow switch operation so fast is in the DOWN position. E8/C. Ran a new track to the 2 pin JST connector from EXT_LA from 10 pin connector on SR input. Added files for E8MX, 2k byte memory expansion board
Parts:
- C1, C2, C3, C4, C5: value (none) -> 47nF; footprint (none) -> Capacitor_THT:C_Disc_D5.0mm_W2.5mm_P5.00mm
- H1, H2: value (none) -> Card_handle; footprint (none) -> EDUC-8:Card_handle
- J1: value (none) -> 32-way-pcb-edge-Educ-8-connectors; footprint (none) -> Connector_PCBEdge:PCB_32pin
- J2: value (none) -> 16-way-pcb-edge-Educ-8-connectors; footprint (none) -> Connector_PCBEdge:PCB_16pin
- J3: value (none) -> Conn_01x01_Male; footprint (none) -> Connector_Pin:Pin_D1.0mm_L10.0mm
- J?: value (none) -> Conn_01x02_Male; footprint (none) -> Connector_JST:JST_XH_S2B-XH-A_1x02_P2.50mm_Horizontal
- J?: value (none) -> Conn_01x03_Male; footprint (none) -> Connector_JST:JST_XH_S3B-XH-A_1x03_P2.50mm_Horizontal
- R1, R2, R3, R4, R5: value (none) -> 820R; footprint (none) -> Resistor_THT:R_Axial_DIN0207_L6.3mm_D2.5mm_P10.16mm_Horizontal
- U1, U10, U11, U12, U5, U6: value (none) -> 7400; footprint (none) -> Package_DIP:DIP-14_W7.62mm
- U1, U10, U11, U12, U5, U6: value (none) -> 7400
- U13, U7: value (none) -> 74LS05; footprint (none) -> Package_DIP:DIP-14_W7.62mm
- U13, U7: value (none) -> 74LS05
- U14, U8: value (none) -> 7496; footprint (none) -> Package_DIP:DIP-16_W7.62mm
- U15, U9: value (none) -> 74LS95; footprint (none) -> Package_DIP:DIP-14_W7.62mm
- U16: value (none) -> 74LS157; footprint (none) -> Package_DIP:DIP-16_W7.62mm
- U17: value (none) -> 74LS04; footprint (none) -> Package_DIP:DIP-14_W7.62mm
- U17: value (none) -> 74LS04
- U18, U19: value (none) -> 74LS01; footprint (none) -> Package_DIP:DIP-14_W7.62mm
- U18, U19: value (none) -> 74LS01
- U2, U3: value (none) -> D2115; footprint (none) -> Package_DIP:DIP-16_W7.62mm
- U4: value (none) -> 74LS93; footprint (none) -> Package_DIP:DIP-14_W7.62mm
