File: 256 word memory/256 word memory.kicad_sch (KiCad schematic)
At the start: 36 parts, among them J1 Conn_01x02_Male, J2 Conn_01x03_Male, J3 16-way-pcb-edge-Educ-8-connec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, J4 Conn_01x01_Male, J5 32-way-pcb-edge-Educ-8-connec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, U1 74LS05, U10 74LS95, U11 7400, U12 7400, U13 74LS93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

Commit message: Changes 20-7-2025 E8/T. Connected 3 missing supply rail tracks to ICS Added flood fill top and bottom to reduce noise E8/F Corrected labelling on RHS board to reflect EXT_LA not GND Changed fast slow switch operation so fast is in the DOWN position. E8/C. Ran a new track to the 2 pin JST connector from EXT_LA from 10 pin connector on SR input. Added files for E8MX, 2k byte memory expansion board
Parts:
- U11, U12, U14, U15, U17, U7: value 7400 -> 74LS00
