File: Accumulator/Accumulator.kicad_sch (KiCad schematic)
At the start: 22 parts, among them J2 16-way-pcb-edge-Educ-8-connec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, U1 74LS95, U10 74LS01, U2 74LS05, U3 74LS95, U4 74LS05, U5 74LS01, U6 74LS04, U7 7400, U8 74LS10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

Commit message: Schematic update 2024-04-14 plus fixes
Parts:
- C4: value (none) -> 47nF; footprint (none) -> Capacitor_THT:C_Rect_L11.0mm_W2.8mm_P10.00mm_MKT
- H1: value Card_handle -> (none); symbol Accumulator-rescue:Card_handle-EDUC-8 -> EDUC8:Card_handle-EDUC-8
- H2: symbol Accumulator-rescue:Card_handle-EDUC-8 -> EDUC8:Card_handle-EDUC-8
- J1: footprint (none) -> Connector_PCBEdge:PCB_16pin; symbol Accumulator-rescue:16-way-pcb-edge-Educ-8-connectors-EDUC-8 -> EDUC8:16-way-pcb-edge-Educ-8-connectors-EDUC-8
- J2: symbol Accumulator-rescue:16-way-pcb-edge-Educ-8-connectors-EDUC-8 -> EDUC8:16-way-pcb-edge-Educ-8-connectors-EDUC-8
- R4: value (none) -> 2K2; footprint (none) -> Resistor_THT:R_Axial_DIN0207_L6.3mm_D2.5mm_P10.16mm_Horizontal
Connections:
- net +5V: now also J1.2, J1.3
- net A-BUS: now also J1.4
- net AC0: now also J1.11, J2.9
- net AC1: now also J2.10
- net AC2: now also J2.11
- net AC3: now also J2.12
- net AC4: now also J2.13
- net AC5: now also J2.14
- net AC6: now also J2.15
- net AC7: now also J2.16
- net AC=0: now also J1.15
- net B-BUS: now also J1.5
- net C-BUS: now also J1.6
- net D-BUS: now also J1.7
- net GND: now also H1.1 (GND), H2.1 (GND), J1.1, J1.16
- net MCP: now also J1.9
- net T1: now also J1.13
- net T2-9: now also J1.12
- net ~{AND}: now also J2.1
- net ~{CLA}: now also J2.8
- net ~{CMA}: now also J2.7
- net ~{DCA}: now also J2.3
- net ~{IAC}: now also J2.5
- net ~{IOT_Shift}: now also J1.10
- net ~{RAL}: now also J2.6
- net ~{RAR}: now also J2.4
- net ~{T13.RAR}: now also J1.8
- net ~{T2-9(TAD+IAC+CMA}): now also J1.14
- net ~{TAD}: now also J2.2
Other:
- note added: "Reference(s) Value C1 47nF C2 47nF C3 47nF C4 47nF H1 Card_handle H2 Card_handle J1 16-way-pcb-edge-Educ-8-connectors J2 16-way-pcb-edge-Educ-8-connectors R1 820 R2 2K2 R3 2K2 R4 2K2 U1 74LS95 U2 74LS05 U3 74LS95 U4 74LS05 U5 74LS01 U6 74LS04 U7 7400 U8 74LS10 U9 7400 U10 74LS01"
- note removed: "0.47uF"
- note removed: "1/4 watt resistor"
- note removed: "2K2"
- note removed: "7400"
- note removed: "7410"
- note removed: "7495"
- note removed: "820R"
- note removed: "C1"
- note removed: "C2"
- note removed: "C3"
- note removed: "C4"
- note removed: "Polyester capacitor"
- note removed: "Quad NAND"
- note removed: "R1"
- note removed: "R2"
- note removed: "R3"
- note removed: "R4"
- note removed: "Triple 3 input NAND"
- note removed: "U1"
- note removed: "U10"
- note removed: "U2"
- note removed: "U3"
- note removed: "U4"
- note removed: "U5"
- note removed: "U6"
- note removed: "U7"
- note removed: "U8"
- note removed: "U9"
- note removed: "shift register"

Commit message: Changes 20-7-2025 E8/T. Connected 3 missing supply rail tracks to ICS Added flood fill top and bottom to reduce noise E8/F Corrected labelling on RHS board to reflect EXT_LA not GND Changed fast slow switch operation so fast is in the DOWN position. E8/C. Ran a new track to the 2 pin JST connector from EXT_LA from 10 pin connector on SR input. Added files for E8MX, 2k byte memory expansion board
Parts:
- H1: value (none) -> Card_handle; symbol EDUC8:Card_handle-EDUC-8 -> Accumulator-rescue:Card_handle-EDUC-8
- H2: symbol EDUC8:Card_handle-EDUC-8 -> Accumulator-rescue:Card_handle-EDUC-8
- J1: value (none) -> 16-way-pcb-edge-Educ-8-connectors; symbol EDUC8:16-way-pcb-edge-Educ-8-connectors-EDUC-8 -> Accumulator-rescue:16-way-pcb-edge-Educ-8-connectors-EDUC-8
- J2: symbol EDUC8:16-way-pcb-edge-Educ-8-connectors-EDUC-8 -> Accumulator-rescue:16-way-pcb-edge-Educ-8-connectors-EDUC-8
Connections:
- net +5V: no longer J1.2, J1.3
- net A-BUS: no longer J1.4
- net AC0: no longer J1.11, J2.9
- net AC1: no longer J2.10
- net AC2: no longer J2.11
- net AC3: no longer J2.12
- net AC4: no longer J2.13
- net AC5: no longer J2.14
- net AC6: no longer J2.15
- net AC7: no longer J2.16
- net AC=0: no longer J1.15
- net B-BUS: no longer J1.5
- net C-BUS: no longer J1.6
- net D-BUS: no longer J1.7
- net GND: no longer H1.1 (GND), H2.1 (GND), J1.1, J1.16
- net MCP: no longer J1.9
- net RAL: now also U6.5
- net T1: no longer J1.13
- net T2-9: no longer J1.12
- net ~{AND}: no longer J2.1
- net ~{CLA}: no longer J2.8
- net ~{CMA}: no longer J2.7
- net ~{DCA}: no longer J2.3
- net ~{IAC}: no longer J2.5
- net ~{RAL}: no longer J2.6
- net ~{RAR}: no longer J2.4
- net ~{T13.RAR}: no longer J1.8
- net ~{T2-9(TAD+IAC+CMA}): no longer J1.14
- net ~{TAD}: no longer J2.2
- net ~{IOT_Shift} renamed IOT_SHIFT
- net IOT_SHIFT: no longer J1.10
- no-connect marks 6 -> 5
Other:
- note added: "0.47uF"
- note added: "1/4 watt resistor"
- note added: "2K2"
- note added: "7400"
- note added: "7410"
- note added: "7495"
- note added: "820R"
- note added: "C1"
- note added: "C2"
- note added: "C3"
- note added: "C4"
- note added: "Polyester capacitor"
- note added: "Quad NAND"
- note added: "R1"
- note added: "R2"
- note added: "R3"
- note added: "R4"
- note added: "Triple 3 input NAND"
- note added: "U1"
- note added: "U10"
- note added: "U2"
- note added: "U3"
- note added: "U4"
- note added: "U5"
- note added: "U6"
- note added: "U7"
- note added: "U8"
- note added: "U9"
- note added: "shift register"
- note removed: "Reference(s) Value C1 47nF C2 47nF C3 47nF C4 47nF H1 Card_handle H2 Card_handle J1 16-way-pcb-edge-Educ-8-connectors J2 16-way-pcb-edge-Educ-8-connectors R1 820 R2 2K2 R3 2K2 R4 2K2 U1 74LS95 U2 74LS05 U3 74LS95 U4 74LS05 U5 74LS01 U6 74LS04 U7 7400 U8 74LS10 U9 7400 U10 74LS01"
- moved on the sheet: U4A
