File: E8Serial/RS232/RS232.kicad_pcb (KiCad board)
At the start: 2 copper layers, 125 x 113 mm, 28 parts, among them J1 DB9_Male, J10 Conn_01x06_Male, J11 Conn_01x06_Male, J5 Conn_01x04_Female, J6 Conn_01x04_Female, J7 Conn_01x04_Female, J9 Conn_01x04_Female, Q1 BC548, Q2 BC548, U1 MAX232

Commit message: Changes 20-7-2025 E8/T. Connected 3 missing supply rail tracks to ICS Added flood fill top and bottom to reduce noise E8/F Corrected labelling on RHS board to reflect EXT_LA not GND Changed fast slow switch operation so fast is in the DOWN position. E8/C. Ran a new track to the 2 pin JST connector from EXT_LA from 10 pin connector on SR input. Added files for E8MX, 2k byte memory expansion board
Parts:
- removed D2: 1N5819, Diode_THT:D_DO-41_SOD81_P10.16mm_Horizontal
- C6, C8: footprint Capacitor_THT:CP_Axial_L11.0mm_D6.0mm_P18.00mm_Horizontal -> Capacitor_THT:CP_Radial_D6.3mm_P2.50mm
- moved C8 13.8 mm to (62.4, 109.4)
- moved J11 5.27 mm to (75.4, 33.8), turned to 0 degrees
- moved J10 5.24 mm to (75.4, 116.8), turned to 0 degrees
Connections:
- J1 pad 1: Net-(J1-Pad1) -> unconnected-(J1-Pad1)
- J1 pad 4: Net-(J1-Pad4) -> unconnected-(J1-Pad4)
- J1 pad 6: Net-(J1-Pad6) -> unconnected-(J1-Pad6)
- J1 pad 9: Net-(J1-Pad9) -> unconnected-(J1-Pad9)
- J10 pad 1: I_data -> I_rst
- J10 pad 3: I_rst -> GND
- J10 pad 4: I_clock -> I_data
- J10 pad 5: Net-(D2-Pad2) -> I_clock
- J10 pad 6: GND -> +5V
- J11 pad 1: data -> rst
- J11 pad 3: rst -> GND
- J11 pad 4: clock -> data
- J11 pad 5: Net-(D2-Pad2) -> clock
- J11 pad 6: GND -> +5V
- U1 pad 10: Net-(U1-Pad10) -> unconnected-(U1-Pad10)
- U1 pad 12: Net-(U1-Pad12) -> RX
- U1 pad 9: Net-(U1-Pad9) -> unconnected-(U1-Pad9)
Routing:
- net Net-(D2-Pad2): track 92.7 -> 0.00 mm
- net RX: track 13.4 -> 60.1 mm
- net Net-(U1-Pad12): track 46.6 -> 0.00 mm
- net clock: track 26.8 -> 9.86 mm
- net I_clock: track 28.1 -> 12.4 mm
- net +5V: track 250.6 -> 261.7 mm
- net I_data: track 11.2 -> 12.6 mm
- net flag: track 9.37 -> 8.81 mm
- net rst: track 9.37 -> 8.81 mm
Other:
- net class Default removed
- board text added: "+5V"
- board text added: "1"
- board text added: "CLOCK"
- board text added: "DATA"
- board text added: "FLAG"
- board text added: "GND"
- board text added: "RST FLAG"
- board text removed: "1 ~DATA 2 ~FLAG 3 ~RESET 4 ~RESET FLAG 5 +5V 6 GND"
