File: EXTENDER CARDS/EXTENDER CARDS.kicad_pcb (KiCad board)
At the start: 2 copper layers, 266 x 180.1 mm, 5 parts, among them J1 32-way-pcb-edge-Educ-8-connec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, J2 36-way-pcb-edge-socket-Educ-8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, J3 16-way-pcb-edge-Educ-8-connec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, J4 36-way-edge-connector-Educ-8-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

Commit message: Changes 20-7-2025 E8/T. Connected 3 missing supply rail tracks to ICS Added flood fill top and bottom to reduce noise E8/F Corrected labelling on RHS board to reflect EXT_LA not GND Changed fast slow switch operation so fast is in the DOWN position. E8/C. Ran a new track to the 2 pin JST connector from EXT_LA from 10 pin connector on SR input. Added files for E8MX, 2k byte memory expansion board
Parts:
- moved J2 74.4 mm to (322.4, 25.8)
- moved J4 74.4 mm to (154.1, 25.8)
- moved J3 57.0 mm to (81.2, 218.7)
- moved J1 57.0 mm to (170.3, 218.6)
- moved REF** 57.0 mm to (71.9, 139.5)
Routing:
- net Net-(J3-Pad15): track 169.0 -> 209.0 mm
- net Net-(J3-Pad13): track 169.0 -> 209.0 mm
- net Net-(J1-Pad32): track 168.9 -> 208.9 mm
- net Net-(J1-Pad9): track 168.9 -> 188.9 mm
- net Net-(J1-Pad6): track 168.9 -> 188.9 mm
- net Net-(J3-Pad8): track 169.0 -> 189.0 mm
- net Net-(J3-Pad7): track 169.0 -> 189.0 mm
- net Net-(J3-Pad6): track 169.0 -> 189.0 mm
- net Net-(J3-Pad4): track 169.0 -> 189.0 mm
- net Net-(J3-Pad3): track 169.0 -> 189.0 mm
- net Net-(J3-Pad2): track 169.0 -> 189.0 mm
- net Net-(J3-Pad16): track 169.0 -> 189.0 mm
- net Net-(J3-Pad14): track 168.1 -> 188.1 mm
- net Net-(J3-Pad12): track 169.0 -> 189.0 mm
- net Net-(J3-Pad10): track 169.0 -> 189.0 mm
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Other:
- board size 266 x 180.1 mm -> 266 x 200.1 mm
- net class Default removed
- board text added: "CAREFULLY CUT A NOTCH BETWEEN 2 PADS TO USE THIS EXTENDER ON BOARDS WITH 2 SHORTER EDGE CONNECTORS. DO NOT CUT THE CONNECTORS!!!!"
