File: PC and ADDER 74LS74 MOD/PC and ADDER 74LS74 MOD.kicad_pcb (KiCad board)
At the start: 2 copper layers, 220 x 160 mm, 30 parts, among them J1 32-way-pcb-edge-Educ-8-connec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, J2 Conn_01x03_Male, J3 Conn_01x03_Male, J4 Conn_01x02_Male, J5 16-way-pcb-edge-Educ-8-connec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, U1 7496, U10 7400, U11 7400, U12 74LS04, U13 74LS20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

Commit message: Changes 20-7-2025 E8/T. Connected 3 missing supply rail tracks to ICS Added flood fill top and bottom to reduce noise E8/F Corrected labelling on RHS board to reflect EXT_LA not GND Changed fast slow switch operation so fast is in the DOWN position. E8/C. Ran a new track to the 2 pin JST connector from EXT_LA from 10 pin connector on SR input. Added files for E8MX, 2k byte memory expansion board
Parts:
- J2, J3: footprint Connector_JST:JST_XH_B3B-XH-AM_1x03_P2.50mm_Vertical -> Connector_JST:JST_XH_S3B-XH-A-1_1x03_P2.50mm_Horizontal
- J4: footprint Connector_JST:JST_XH_B2B-XH-AM_1x02_P2.50mm_Vertical -> Connector_JST:JST_XH_S2B-XH-A_1x02_P2.50mm_Horizontal
- U10, U11, U6, U7: value 7400 -> 74LS00
Other:
- board text added: "50 YEARS"
