File: PC and ADDER 74LS74 MOD/PC and ADDER 74LS74 MOD.kicad_sch (KiCad schematic)
At the start: 28 parts, among them J1 32-way-pcb-edge-Educ-8-connec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, J2 Conn_01x03_Male, J3 Conn_01x03_Male, J4 Conn_01x02_Male, J5 16-way-pcb-edge-Educ-8-connec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, U1 7496, U10 7400, U11 7400, U12 74LS04, U13 74LS20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

Commit message: Changes 20-7-2025 E8/T. Connected 3 missing supply rail tracks to ICS Added flood fill top and bottom to reduce noise E8/F Corrected labelling on RHS board to reflect EXT_LA not GND Changed fast slow switch operation so fast is in the DOWN position. E8/C. Ran a new track to the 2 pin JST connector from EXT_LA from 10 pin connector on SR input. Added files for E8MX, 2k byte memory expansion board
Parts:
- U10, U11, U6, U7: value 7400 -> 74LS00
Other:
- note added: "C1 47nF C2 47nF C3 47nF C4 47nF C5 47nF C6 47nF H1 Card_handle H2 Card_handle J1 32-way-pcb-edge-Educ-8-connectors J2 Conn_01x03_Male J3 Conn_01x03_Male J4 Conn_01x02_Male J5 16-way-pcb-edge-Educ-8-connectors R1 2k2 R2 2k2 U1 7496 U2 7496 U3 74LS10 U4 74LS74 U5 74LS10 U6 74LS00 U7 74LS00 U8 7480 or 74LS80 U9 74LS04 U10 74LS00 U11 74LS00 U12 74LS04 U13 74LS20 U14 74LS01"
- note removed: "C1 47nF C2 47nF C3 47nF C4 47nF C5 47nF C6 47nF H1 Card_handle H2 Card_handle J1 32-way-pcb-edge-Educ-8-connectors J2 Conn_01x03_Male J3 Conn_01x03_Male J4 Conn_01x02_Male J5 16-way-pcb-edge-Educ-8-connectors R1 2k2 R2 2k2 U1 7496 U2 7496 U3 74LS10 U4 74LS74 U5 74LS10 U6 7400 U7 7400 U8 7480 U9 74LS04 U10 7400 U11 7400 U12 74LS04 U13 74LS20 U14 74LS01"
