File: Power Supply/EDUC-8 PSU.kicad_pcb (KiCad board)
At the start: 2 copper layers, 125 x 116.8 mm, 43 parts, among them J1 Conn_01x01_Male, J10 +5V, J11 GND, J2 Conn_01x01_Male, J4 Conn_01x01_Male, J5 Conn_01x01_Male, J6 Conn_01x01_Male, J7 Conn_01x01_Male, J8 Conn_01x01_Male, J9 DC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

Commit message: Changes 20-7-2025 E8/T. Connected 3 missing supply rail tracks to ICS Added flood fill top and bottom to reduce noise E8/F Corrected labelling on RHS board to reflect EXT_LA not GND Changed fast slow switch operation so fast is in the DOWN position. E8/C. Ran a new track to the 2 pin JST connector from EXT_LA from 10 pin connector on SR input. Added files for E8MX, 2k byte memory expansion board
Parts:
- C8: value 470uF 10V -> 470uF 35V
- D5: value 5.6V -> 6.2V
- moved J10 106.5 mm to (171.4, 135.6), turned to -90 degrees
- moved J11 106.2 mm to (171.1, 49.9), turned to -90 degrees
- moved J9 105.9 mm to (171.1, 71.6), turned to -90 degrees
- moved C7 70.6 mm to (162.9, 129.4)
- moved Q3 69.3 mm to (157.7, 118.3), turned to 0 degrees
- moved F1 66.5 mm to (73.8, 85.8)
- moved REF** 66.5 mm to (72.4, 143.7)
- moved C1 66.5 mm to (102.4, 120.2)
- moved C2 66.5 mm to (72.4, 120.3)
- moved C5 66.5 mm to (170.7, 78.4)
- moved C6 66.5 mm to (125.4, 78.3)
- moved D1 66.5 mm to (71.3, 108.1)
- moved D2 66.5 mm to (78.9, 108.1)
- moved D3 66.5 mm to (64.0, 92.9)
- moved D4 66.5 mm to (56.4, 92.9)
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Routing:
- net Net-(C1-Pad1): track 168.7 -> 439.1 mm
- net +5V: track 45.9 -> 287.3 mm
- net Net-(Q4-Pad2): track 0.00 -> 54.7 mm
- net GND: track 65.0 -> 115.2 mm
- net Net-(Q4-Pad1): track 5.90 -> 42.0 mm
- net Net-(C7-Pad1): track 45.4 -> 75.0 mm
- net Net-(C8-Pad1): track 0.00 -> 26.4 mm
- net Net-(D5-Pad1): track 0.00 -> 10.5 mm
- net Net-(C7-Pad2): track 0.00 -> 10.1 mm
- net Net-(Q2-Pad2): track 37.6 -> 41.0 mm
- net Net-(Q1-Pad2): track 37.5 -> 40.5 mm
- net Net-(Q4-Pad3): track 2.73 -> 0.00 mm
- added copper zone on B.Cu, net GND
Other:
- board text added: "2A Fast"
- board text removed: "3A Fast"
