File: Power Supply/EDUC-8 PSU.kicad_sch (KiCad schematic)
At the start: 42 parts, among them J1 Conn_01x01_Male, J10 +5V, J11 GND, J2 Conn_01x01_Male, J3 Conn_01x01_Male, J4 Conn_01x01_Male, J5 Conn_01x01_Male, J6 Conn_01x01_Male, J7 Conn_01x01_Male, J8 Conn_01x01_Male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

Commit message: Changes 20-7-2025 E8/T. Connected 3 missing supply rail tracks to ICS Added flood fill top and bottom to reduce noise E8/F Corrected labelling on RHS board to reflect EXT_LA not GND Changed fast slow switch operation so fast is in the DOWN position. E8/C. Ran a new track to the 2 pin JST connector from EXT_LA from 10 pin connector on SR input. Added files for E8MX, 2k byte memory expansion board
Other:
- note added: "C1 4700uF C2 4700uF C5 47nF C6 47nF C7 22nF C8 470uF 10V D1 1N5404 D2 1N5404 D3 1N5404 D4 1N5404 D5 5.6V F1 Fuse J1 PCB QC connector J2 PCB QC connector J3 PCB QC connector J4 PCB QC connector J5 PCB QC connector J6 PCB QC connector J7 PCB QC connector J8 PCB QC connector J9 DC J10 +5V J11 GND Q1 2N3055 Q2 2N3055 Q3 2N4037 Q4 BC108 Q5 BC108 R1 10R R2 10R R3 0.33R R4 0.33R R5 100R R6 100R R7 120R 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"
- moved on the sheet: C1, C2, C5, C6, C7, C8, D1, D2, D3, D4, D5, F1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
