File: Power Supply/Crowbar/EDUC-8 Crowbar/EDUC-8 Crowbar.kicad_pcb (KiCad board)
At the start: 2 copper layers, 99 x 27 mm, 11 parts, among them J1 +5V, J2 DC, J3 GND, J4 FAN+, J5 FAN-, Q1 TIC106, Q2 TIC106

Commit message: Changes 20-7-2025 E8/T. Connected 3 missing supply rail tracks to ICS Added flood fill top and bottom to reduce noise E8/F Corrected labelling on RHS board to reflect EXT_LA not GND Changed fast slow switch operation so fast is in the DOWN position. E8/C. Ran a new track to the 2 pin JST connector from EXT_LA from 10 pin connector on SR input. Added files for E8MX, 2k byte memory expansion board
Other:
- net class Default removed
