File: Timing/educ 8 timing .kicad_pcb (KiCad board)
At the start: 4 copper layers, 220 x 159.9 mm, 45 parts, among them J1 32-way-pcb-edge-Educ-8-connec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, J2 CLK, J3 ~RST, Q1 BC108, U1 74LS20, U10 74LS00, U11 74154, U12 74LS73, U13 74LS00, U14 74LS73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

Commit message: Changes 20-7-2025 E8/T. Connected 3 missing supply rail tracks to ICS Added flood fill top and bottom to reduce noise E8/F Corrected labelling on RHS board to reflect EXT_LA not GND Changed fast slow switch operation so fast is in the DOWN position. E8/C. Ran a new track to the 2 pin JST connector from EXT_LA from 10 pin connector on SR input. Added files for E8MX, 2k byte memory expansion board
Parts:
- added J4: Conn_01x03_Male, Connector_JST:JST_XH_B3B-XH-A_1x03_P2.50mm_Vertical, F.Cu at (224.2, 96.8)
- C10: value 47nF -> 100nF; footprint Capacitor_THT:C_Disc_D7.0mm_W2.5mm_P5.00mm -> Capacitor_THT:C_Disc_D5.0mm_W2.5mm_P5.00mm
- C3, C6, C9: value 1uF -> 100nF; footprint Capacitor_THT:C_Axial_L5.1mm_D3.1mm_P12.50mm_Horizontal -> Capacitor_THT:C_Disc_D5.0mm_W2.5mm_P5.00mm
- C4, C5, C7, C8: value 47nF -> 100nF
- Q1: value BC108 -> BC548; footprint Package_TO_SOT_THT:TO-18-3 -> Package_TO_SOT_THT:TO-92_Wide
- U2: value 7400 -> 74LS00
- moved C3 78.5 mm to (33.4, 53.5)
- moved C6 74.7 mm to (34.0, 127.9)
- moved C9 7.52 mm to (34.0, 106.0)
- moved Q1 3.98 mm to (227.2, 46.4), turned to 90 degrees
Connections:
- Q1 pad 1: Net-(Q1-Pad1) -> +5V
- Q1 pad 3: +5V -> Net-(Q1-E)
- R2 pad 1: Net-(Q1-Pad1) -> Net-(Q1-E)
- U6 pad 4: Net-(Q1-Pad1) -> Net-(Q1-E)
Routing:
- net ~{RUN}: track 207.1 -> 238.0 mm, vias 4 -> 5
- net +5V: track 909.6 -> 940.5 mm
- net Net-(Q1-E): track 0.00 -> 28.6 mm
- net Net-(Q1-Pad1): track 27.4 -> 0.00 mm
- net ~{RST}: track 467.7 -> 488.2 mm
- net GND: track 666.1 -> 658.1 mm
- net ~{DEP+EXM}: track 326.5 -> 329.6 mm
- net Net-(U1-Pad9): track 229.6 -> 231.0 mm
- net FAST_SLOW: track 175.7 -> 174.5 mm
- net MB4: track 246.8 -> 246.0 mm
- added copper zone on F.Cu, net GND
Other:
- board text added: "50 YEARS"
- board text added: "Designed by Jamieson Rowe 1974 Electronics Australia PCB by Gwyllym Suter 2024"
- board text added: "TO E8/MX"
- board text removed: "Designed by Jamieson Rowe 1974 Electronics Australia PCB by Gwyllym Suter 2022"
- board text removed: "V1.1"
