File: Timing/educ 8 timing .kicad_sch (KiCad schematic)
At the start: 44 parts, among them J1 32-way-pcb-edge-Educ-8-connec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, J2 CLK, J3 ~RST, Q1 BC108, U1 74LS20, U10 7400, U11 74154, U12 74LS73, U13 7400, U14 74LS73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

Commit message: Schematic update 2024-04-14 plus fixes
Other:
- note added: "C1 220pF C2 47uF C3 47nF C4 47nF C5 47nF C6 1uF C7 47nF C8 47nF C9 1uF C10 47nF H1 Card_handle H2 Card_handle J1 32-way-pcb-edge J2 CLK J3 ~RST Q1 BC108 R1 2k2 R2 470R R3 10k R4 2K2 R5 100K R6 2k2 R7 2k2 U1 74LS20 U2 74LS00 U3 74LS04 U4 74LS10 U5 74LS161 U6 74LS13 U7 74LS00 U8 74LS00 U9 74LS00 U10 74LS00 U11 74154 U12 74LS73 U13 74LS00 U14 74LS73 U15 74LS04 U16 74LS00 U17 74LS04 U18 74LS00 U19 74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"
- note added: "TIMING"
- note removed: "1 of 16 binary decoder"
- note removed: "4Bit binary counter with ripple carry"
- note removed: "7400"
- note removed: "7404"
- note removed: "7410"
- note removed: "7413"
- note removed: "74154"
- note removed: "74161"
- note removed: "7473"
- note removed: "74LS20"
- note removed: "9311"
- note removed: "9316"
- note removed: "BC108"
- note removed: "BC548"
- note removed: "Description"
- note removed: "Dual 4 input NAND"
- note removed: "Dual 4 input NAND, open collector"
- note removed: "Dual J/K flip flow with clear"
- note removed: "Gate"
- note removed: "Hex Inverter"
- note removed: "NPN signal transistor"
- note removed: "Part No"
- note removed: "Q1"
- note removed: "Quad 2 input NAND"
- note removed: "RefDes"
- note removed: "Substitute"
- note removed: "Triple 3 input NAND"
- note removed: "U1"
- note removed: "U10"
- note removed: "U11"
- note removed: "U12"
- note removed: "U13"
- note removed: "U14"
- note removed: "U15"
- note removed: "U16"
- note removed: "U17"
- note removed: "U18"
- note removed: "U19"
- note removed: "U2"
- note removed: "U20"
- note removed: "U21"
- note removed: "U3"
- note removed: "U4"
- note removed: "U5"
- note removed: "U6"
- note removed: "U7"
- note removed: "U8"
- note removed: "U9"
- note removed: "“"

Commit message: Changes 20-7-2025 E8/T. Connected 3 missing supply rail tracks to ICS Added flood fill top and bottom to reduce noise E8/F Corrected labelling on RHS board to reflect EXT_LA not GND Changed fast slow switch operation so fast is in the DOWN position. E8/C. Ran a new track to the 2 pin JST connector from EXT_LA from 10 pin connector on SR input. Added files for E8MX, 2k byte memory expansion board
Parts:
- removed Q1: BC108, Package_TO_SOT_THT:TO-18-3, symbol Transistor_BJT:BC108
- added J4: Conn_01x03_Male, Connector_JST:JST_XH_B3B-XH-A_1x03_P2.50mm_Vertical, symbol Connector:Conn_01x03_Male
- added Q1: BC548, Package_TO_SOT_THT:TO-92_Wide, symbol Transistor_BJT:BC548
- C10: value 47nF -> 100nF; footprint Capacitor_THT:C_Disc_D7.0mm_W2.5mm_P5.00mm -> Capacitor_THT:C_Disc_D5.0mm_W2.5mm_P5.00mm
- C3: value 47nF -> 100nF; footprint Capacitor_THT:C_Axial_L5.1mm_D3.1mm_P12.50mm_Horizontal -> Capacitor_THT:C_Disc_D5.0mm_W2.5mm_P5.00mm
- C4, C5, C7, C8: value 47nF -> 100nF
- C6, C9: value 1uF -> 100nF; footprint Capacitor_THT:C_Axial_L5.1mm_D3.1mm_P12.50mm_Horizontal -> Capacitor_THT:C_Disc_D5.0mm_W2.5mm_P5.00mm
- U10, U13, U16, U18, U2, U21, U7, U8, U9: value 7400 -> 74LS00
Connections:
- net +5V: now also Q1.1 (C)
- net FAST_SLOW: now also Q1.2 (B)
- net GND: now also J4.1 (Pin_1)
- net ~{RST}: now also J4.3 (Pin_3)
- net ~{RUN}: now also J4.2 (Pin_2)
- net at R2.1, U6.4: now also Q1.3 (E)
Other:
- note added: "C1 220pF C2 47uF C3 47nF C4 47nF C5 47nF C6 1uF C7 47nF C8 47nF C9 1uF C10 47nF H1 Card_handle H2 Card_handle J1 32-way-pcb-edge J2 CLK J3 ~RST J4 JST_XH_02 Q1 BC548 R1 2k2 R2 470R R3 10k R4 2K2 R5 100K R6 2k2 R7 2k2 U1 74LS20 U2 74LS00 U3 74LS04 U4 74LS10 U5 74LS161 U6 74LS13 U7 74LS00 U8 74LS00 U9 74LS00 U10 74LS00 U11 74154 or 74LS154 U12 74LS73 U13 74LS00 U14 74LS73 U15 74LS04 U16 74LS00 U17 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"
- note removed: "C1 220pF C2 47uF C3 47nF C4 47nF C5 47nF C6 1uF C7 47nF C8 47nF C9 1uF C10 47nF H1 Card_handle H2 Card_handle J1 32-way-pcb-edge J2 CLK J3 ~RST Q1 BC108 R1 2k2 R2 470R R3 10k R4 2K2 R5 100K R6 2k2 R7 2k2 U1 74LS20 U2 74LS00 U3 74LS04 U4 74LS10 U5 74LS161 U6 74LS13 U7 74LS00 U8 74LS00 U9 74LS00 U10 74LS00 U11 74154 U12 74LS73 U13 74LS00 U14 74LS73 U15 74LS04 U16 74LS00 U17 74LS04 U18 74LS00 U19 74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"
- note removed: "swap pin 8,9"
