File: 128 X 16 RAM V5 FINAL/128 X 16 RAM V4 FINAL .kicad_sch (KiCad schematic)
At the start: 112 parts, among them J1 Conn_02x08_Counter_Clockwise, J11 Conn_01x02, J2 Conn_01x03_Pin, J3 DB25_Pins, J4 Conn_01x10, J5 Input, J6 Conn_01x02, J7 Output, U1 D2115, U10 D2115, U11 D2115, U12 D2115, U13 D2115, U14 D2115, U15 D2115, U16 D2115, U18 74LS138, U19 4017, U2 D2115, U20 74LS138, U21 74LS07, U22 74LS157, U23 74LS541, U24 74LS04, U25 74LS123, U26 74LS00, U27 74LS595, U3 D2115, U4 D2115, U5 D2115, U6 D2115, U7 D2115, U8 D2115, U9 D2115

Commit message: 128x16 RAM V5 update
Parts:
- removed unit 5 of U24
- added D22: BAT48, Diode_THT:D_DO-35_SOD27_P7.62mm_Horizontal, symbol Diode:BAT48RL
- C19, C20: value 220pF -> 1nF
- U27: footprint (none) -> Package_DIP:DIP-16_W7.62mm
Connections:
- net ~{RUN} is gone; now on net ~{DEP+LA}: J2.2 (Pin_2)
- net +5V: now also U25.10 (B)
- net Latch Bank: now also D22.2 (A)
- net at D17.1 (K), D18.1 (K), R27.1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: now also D22.1 (K)
- net at U25.4 (~{Q}): no longer U25.10 (B)
- net ~{DEP+LA}: now reaches U22.1 (S)
Other:
- note added: "CONNECT TO ~{DEP+LA} ON E8/T"
- note added: "When ~{DEP}+~{LA} goes low on the timer board it disables the EXTERNAL PROGRAMMING INTERFACE. used to select BANK 0-15"
- note removed: "CONNECT TO RUN ON E8/T"
- note removed: "U2B is triggerer either by U2A at the end of of set RAM bank escape sequence or by clock pulses to an O/P device."
- note removed: "When ~{RUN} goes low on the timer board it disables the EXTERNAL PROGRAMMING INTERFACE. used to BANK 0-15"
- moved on the sheet: D18, R27
